File: hardware/TEMP_SENSOR.sch (KiCad schematic (older format))
At the start: 8 parts

Commit message: after DRC,
Parts:
- gave numbers to parts that had none: 8
Changed lines of the file:
@@
 $EndBitmap
 $Comp
-L taobao-components:LM75 U?
+L taobao-components:LM75 U1
 U 1 1 5CEF6143
 P 3850 2650
-AR Path="/5CF23B0A/5CEF6143" Ref="U?"  Part="1"
+AR Path="/5CF23B0A/5CEF6143" Ref="U1"  Part="1"
 AR Path="/5D003BDB/5CEF6143" Ref="U?"  Part="1"
 AR Path="/5D003BEA/5CEF6143" Ref="U?"  Part="1"
 AR Path="/5D004194/5CEF6143" Ref="U?"  Part="1"
 AR Path="/5D0041A3/5CEF6143" Ref="U?"  Part="1"
-F 0 "U?" H 3850 3100 50  0000 C CNN
+F 0 "U1" H 3850 3100 50  0000 C CNN
 F 1 "LM75" H 3850 3000 50  0000 C CNN
 F 2 "Package_SO:SOP-8_3.76x4.96mm_P1.27mm" H 3850 2050 50  0001 C CNN
@@
 $EndComp
 $Comp
-L taobao-c:C103,0603 C?
+L taobao-c:C103,0603 C1
 U 1 1 5CEF7ED4
 P 4700 2850
-AR Path="/5CF23B0A/5CEF7ED4" Ref="C?"  Part="1"
+AR Path="/5CF23B0A/5CEF7ED4" Ref="C1"  Part="1"
 AR Path="/5D003BDB/5CEF7ED4" Ref="C?"  Part="1"
 AR Path="/5D003BEA/5CEF7ED4" Ref="C?"  Part="1"
 AR Path="/5D004194/5CEF7ED4" Ref="C?"  Part="1"
 AR Path="/5D0041A3/5CEF7ED4" Ref="C?"  Part="1"
-F 0 "C?" H 4800 2900 50  0000 L CNN
+F 0 "C1" H 4800 2900 50  0000 L CNN
 F 1 "C103,0603" H 4800 2850 50  0000 L CNN
 F 2 "Capacitor_SMD:C_0603_1608Metric_Pad1.05x0.95mm_HandSolder" H 4700 2850 50  0001 C CNN
@@
 $EndComp
 $Comp
-L power:GND #PWR?
+L power:GND #PWR06
 U 1 1 5CEF86F3
 P 4500 3000
-AR Path="/5CF23B0A/5CEF86F3" Ref="#PWR?"  Part="1"
+AR Path="/5CF23B0A/5CEF86F3" Ref="#PWR06"  Part="1"
 AR Path="/5D003BDB/5CEF86F3" Ref="#PWR?"  Part="1"
 AR Path="/5D003BEA/5CEF86F3" Ref="#PWR?"  Part="1"
 AR Path="/5D004194/5CEF86F3" Ref="#PWR?"  Part="1"
 AR Path="/5D0041A3/5CEF86F3" Ref="#PWR?"  Part="1"
-F 0 "#PWR?" H 4500 2750 50  0001 C CNN
+F 0 "#PWR06" H 4500 2750 50  0001 C CNN
 F 1 "GND" H 4550 2800 50  0000 C CNN
 F 2 "" H 4500 3000 50  0001 C CNN
@@
 	4500 2800 4500 3000
 $Comp
-L power:GND #PWR?
+L power:GND #PWR07
 U 1 1 5CEF9E27
 P 4700 3100
-AR Path="/5CF23B0A/5CEF9E27" Ref="#PWR?"  Part="1"
+AR Path="/5CF23B0A/5CEF9E27" Ref="#PWR07"  Part="1"
 AR Path="/5D003BDB/5CEF9E27" Ref="#PWR?"  Part="1"
 AR Path="/5D003BEA/5CEF9E27" Ref="#PWR?"  Part="1"
 AR Path="/5D004194/5CEF9E27" Ref="#PWR?"  Part="1"
 AR Path="/5D0041A3/5CEF9E27" Ref="#PWR?"  Part="1"
-F 0 "#PWR?" H 4700 2850 50  0001 C CNN
+F 0 "#PWR07" H 4700 2850 50  0001 C CNN
 F 1 "GND" H 4750 2900 50  0000 C CNN
 F 2 "" H 4700 3100 50  0001 C CNN
@@
 	4700 2950 4700 3100
 $Comp
-L power:+3V3 #PWR?
+L power:+3V3 #PWR02
 U 1 1 5CEFBBD2
 P 4700 1950
-AR Path="/5CF23B0A/5CEFBBD2" Ref="#PWR?"  Part="1"
+AR Path="/5CF23B0A/5CEFBBD2" Ref="#PWR02"  Part="1"
 AR Path="/5D003BDB/5CEFBBD2" Ref="#PWR?"  Part="1"
 AR Path="/5D003BEA/5CEFBBD2" Ref="#PWR?"  Part="1"
 AR Path="/5D004194/5CEFBBD2" Ref="#PWR?"  Part="1"
 AR Path="/5D0041A3/5CEFBBD2" Ref="#PWR?"  Part="1"
-F 0 "#PWR?" H 4700 1800 50  0001 C CNN
+F 0 "#PWR02" H 4700 1800 50  0001 C CNN
 F 1 "+3V3" H 4750 2150 50  0000 C CNN
 F 2 "" H 4700 1950 50  0001 C CNN
@@
 $EndComp
 $Comp
-L power:GND #PWR?
+L power:GND #PWR05
 U 1 1 5CF0201D
 P 3350 3000
-AR Path="/5CF23B0A/5CF0201D" Ref="#PWR?"  Part="1"
+AR Path="/5CF23B0A/5CF0201D" Ref="#PWR05"  Part="1"
 AR Path="/5D003BDB/5CF0201D" Ref="#PWR?"  Part="1"
 AR Path="/5D003BEA/5CF0201D" Ref="#PWR?"  Part="1"
 AR Path="/5D004194/5CF0201D" Ref="#PWR?"  Part="1"
 AR Path="/5D0041A3/5CF0201D" Ref="#PWR?"  Part="1"
-F 0 "#PWR?" H 3350 2750 50  0001 C CNN
+F 0 "#PWR05" H 3350 2750 50  0001 C CNN
 F 1 "GND" H 3400 2800 50  0000 C CNN
 F 2 "" H 3350 3000 50  0001 C CNN
@@
 	3350 2800 3450 2800
 $Comp
-L Jumper:SolderJumper_2_Open JP?
+L Jumper:SolderJumper_2_Open JP1
 U 1 1 5CF0F377
 P 4700 2200
-AR Path="/5CF23B0A/5CF0F377" Ref="JP?"  Part="1"
+AR Path="/5CF23B0A/5CF0F377" Ref="JP1"  Part="1"
 AR Path="/5D003BDB/5CF0F377" Ref="JP?"  Part="1"
 AR Path="/5D003BEA/5CF0F377" Ref="JP?"  Part="1"
 AR Path="/5D004194/5CF0F377" Ref="JP?"  Part="1"
 AR Path="/5D0041A3/5CF0F377" Ref="JP?"  Part="1"
-F 0 "JP?" V 4654 2268 50  0000 L CNN
+F 0 "JP1" V 4654 2268 50  0000 L CNN
 F 1 "LM75_EN" V 4745 2268 50  0000 L CNN
 F 2 "Jumper:SolderJumper-2_P1.3mm_Open_RoundedPad1.0x1.5mm" H 4700 2200 50  0001 C CNN
@@
 AR Path="/5CF23B4E/5CF66B48" Ref="#PWR?"  Part="1"
 AR Path="/5CF23C1A/5CF66B48" Ref="#PWR?"  Part="1"
-AR Path="/5CF23B0A/5CF66B48" Ref="#PWR?"  Part="1"
+AR Path="/5CF23B0A/5CF66B48" Ref="#PWR01"  Part="1"
 AR Path="/5D003BDB/5CF66B48" Ref="#PWR?"  Part="1"
 AR Path="/5D003BEA/5CF66B48" Ref="#PWR?"  Part="1"
 AR Path="/5D004194/5CF66B48" Ref="#PWR?"  Part="1"
 AR Path="/5D0041A3/5CF66B48" Ref="#PWR?"  Part="1"
-F 0 "#PWR?" H 2350 1100 50  0001 C CNN
+F 0 "#PWR01" H 2350 1100 50  0001 C CNN
 F 1 "+3V3" H 2350 1450 50  0000 C CNN
 F 2 "" H 2350 1250 50  0001 C CNN
@@
 $EndComp
 $Comp
-L taobao-r:R473,0603 R?
+L taobao-r:R473,0603 R1
 U 1 1 5CF6A17C
 P 1800 1250
-AR Path="/5CF23B0A/5CF6A17C" Ref="R?"  Part="1"
+AR Path="/5CF23B0A/5CF6A17C" Ref="R1"  Part="1"
 AR Path="/5D003BDB/5CF6A17C" Ref="R?"  Part="1"
 AR Path="/5D003BEA/5CF6A17C" Ref="R?"  Part="1"
 AR Path="/5D004194/5CF6A17C" Ref="R?"  Part="1"
 AR Path="/5D0041A3/5CF6A17C" Ref="R?"  Part="1"
-F 0 "R?" V 1604 1250 50  0000 C CNN
+F 0 "R1" V 1604 1250 50  0000 C CNN
 F 1 "R473,0603" V 1695 1250 50  0000 C CNN
 F 2 "Resistor_SMD:R_0603_1608Metric_Pad1.05x0.95mm_HandSolder" H 1800 1250 50  0001 C CNN
@@
 $EndComp
 $Comp
-L taobao-r:R473,0603 R?
+L taobao-r:R473,0603 R2
 U 1 1 5CF6A570
 P 1800 1350
-AR Path="/5CF23B0A/5CF6A570" Ref="R?"  Part="1"
+AR Path="/5CF23B0A/5CF6A570" Ref="R2"  Part="1"
 AR Path="/5D003BDB/5CF6A570" Ref="R?"  Part="1"
 AR Path="/5D003BEA/5CF6A570" Ref="R?"  Part="1"
 AR Path="/5D004194/5CF6A570" Ref="R?"  Part="1"
 AR Path="/5D0041A3/5CF6A570" Ref="R?"  Part="1"
-F 0 "R?" V 1904 1350 50  0000 C CNN
+F 0 "R2" V 1904 1350 50  0000 C CNN
 F 1 "R473,0603" V 1995 1350 50  0000 C CNN
 F 2 "Resistor_SMD:R_0603_1608Metric_Pad1.05x0.95mm_HandSolder" H 1800 1350 50  0001 C CNN
@@
 	2800 2300 3050 2300
 $Comp
-L power:GND #PWR?
+L power:GND #PWR04
 U 1 1 5CF08421
 P 3200 2150
-AR Path="/5CF23B0A/5CF08421" Ref="#PWR?"  Part="1"
+AR Path="/5CF23B0A/5CF08421" Ref="#PWR04"  Part="1"
 AR Path="/5D003BDB/5CF08421" Ref="#PWR?"  Part="1"
 AR Path="/5D003BEA/5CF08421" Ref="#PWR?"  Part="1"
 AR Path="/5D004194/5CF08421" Ref="#PWR?"  Part="1"
 AR Path="/5D0041A3/5CF08421" Ref="#PWR?"  Part="1"
-F 0 "#PWR?" H 3200 1900 50  0001 C CNN
+F 0 "#PWR04" H 3200 1900 50  0001 C CNN
 F 1 "GND" H 3122 2113 50  0000 R CNN
 F 2 "" H 3200 2150 50  0001 C CNN
@@
 $EndComp
 $Comp
-L power:+3V3 #PWR?
+L power:+3V3 #PWR03
 U 1 1 5CF08014
 P 3050 2100
-AR Path="/5CF23B0A/5CF08014" Ref="#PWR?"  Part="1"
+AR Path="/5CF23B0A/5CF08014" Ref="#PWR03"  Part="1"
 AR Path="/5D003BDB/5CF08014" Ref="#PWR?"  Part="1"
 AR Path="/5D003BEA/5CF08014" Ref="#PWR?"  Part="1"
 AR Path="/5D004194/5CF08014" Ref="#PWR?"  Part="1"
 AR Path="/5D0041A3/5CF08014" Ref="#PWR?"  Part="1"
-F 0 "#PWR?" H 3050 1950 50  0001 C CNN
+F 0 "#PWR03" H 3050 1950 50  0001 C CNN
 F 1 "+3V3" H 3065 2273 50  0000 C CNN
 F 2 "" H 3050 2100 50  0001 C CNN
@@
 $EndComp
 $Comp
-L Connector:Conn_01x05_Female J?
+L Connector:Conn_01x05_Female J1
 U 1 1 5CF06FB7
 P 2600 2500
-AR Path="/5CF23B0A/5CF06FB7" Ref="J?"  Part="1"
+AR Path="/5CF23B0A/5CF06FB7" Ref="J1"  Part="1"
 AR Path="/5D003BDB/5CF06FB7" Ref="J?"  Part="1"
 AR Path="/5D003BEA/5CF06FB7" Ref="J?"  Part="1"
 AR Path="/5D004194/5CF06FB7" Ref="J?"  Part="1"
 AR Path="/5D0041A3/5CF06FB7" Ref="J?"  Part="1"
-F 0 "J?" H 2492 2885 50  0000 C CNN
+F 0 "J1" H 2492 2885 50  0000 C CNN
 F 1 "LM75_HEADER" H 2492 2794 50  0000 C CNN
 F 2 "Connector_PinHeader_1.27mm:PinHeader_1x05_P1.27mm_Vertical" H 2600 2500 50  0001 C CNN
@@
 P 5450 3100
 AR Path="/5CF23B4E/5CFBC7CB" Ref="#PWR?"  Part="1"
-AR Path="/5CF23B0A/5CFBC7CB" Ref="#PWR?"  Part="1"
+AR Path="/5CF23B0A/5CFBC7CB" Ref="#PWR08"  Part="1"
 AR Path="/5D003BDB/5CFBC7CB" Ref="#PWR?"  Part="1"
 AR Path="/5D003BEA/5CFBC7CB" Ref="#PWR?"  Part="1"
 AR Path="/5D004194/5CFBC7CB" Ref="#PWR?"  Part="1"
 AR Path="/5D0041A3/5CFBC7CB" Ref="#PWR?"  Part="1"
-F 0 "#PWR?" H 5450 2850 50  0001 C CNN
+F 0 "#PWR08" H 5450 2850 50  0001 C CNN
 F 1 "GND" H 5500 2900 50  0000 C CNN
 F 2 "" H 5450 3100 50  0001 C CNN
@@
 P 5450 2700
 AR Path="/5CF23B4E/5CFBC7D3" Ref="R?"  Part="1"
-AR Path="/5CF23B0A/5CFBC7D3" Ref="R?"  Part="1"
+AR Path="/5CF23B0A/5CFBC7D3" Ref="R3"  Part="1"
 AR Path="/5D003BDB/5CFBC7D3" Ref="R?"  Part="1"
 AR Path="/5D003BEA/5CFBC7D3" Ref="R?"  Part="1"
 AR Path="/5D004194/5CFBC7D3" Ref="R?"  Part="1"
 AR Path="/5D0041A3/5CFBC7D3" Ref="R?"  Part="1"
-F 0 "R?" H 5509 2746 50  0000 L CNN
+F 0 "R3" H 5509 2746 50  0000 L CNN
 F 1 "R511,0603" H 5509 2655 50  0000 L CNN
 F 2 "Resistor_SMD:R_0603_1608Metric_Pad1.05x0.95mm_HandSolder" H 5450 2700 50  0001 C CNN
@@
 P 5450 2950
 AR Path="/5CF23B4E/5CFBC7D9" Ref="D?"  Part="1"
-AR Path="/5CF23B0A/5CFBC7D9" Ref="D?"  Part="1"
+AR Path="/5CF23B0A/5CFBC7D9" Ref="D1"  Part="1"
 AR Path="/5D003BDB/5CFBC7D9" Ref="D?"  Part="1"
 AR Path="/5D003BEA/5CFBC7D9" Ref="D?"  Part="1"
 AR Path="/5D004194/5CFBC7D9" Ref="D?"  Part="1"
 AR Path="/5D0041A3/5CFBC7D9" Ref="D?"  Part="1"
-F 0 "D?" V 5496 2882 50  0000 R CNN
+F 0 "D1" V 5496 2882 50  0000 R CNN
 F 1 "LED_GREEN,0603" V 5405 2882 50  0000 R CNN
 F 2 "footprint-lib:LED_0603_1608Metric" V 5450 2950 50  0001 C CNN
