File: hardware/digital_input.sch (KiCad schematic (older format))
At the start: 13 parts

Commit message: after DRC,
Parts:
- added R36: R104,0603, Resistor_SMD:R_0603_1608Metric_Pad1.05x0.95mm_HandSolder, symbol taobao-r:R104,0603
- gave numbers to parts that had none: 13
Connections:
- net +3V3: now also R36.1
- net INT: now also R36.2
