File: hardware/esp12_user_button.sch (KiCad schematic (older format))
At the start: 6 parts

Commit message: after DRC,
Parts:
- gave numbers to parts that had none: 6
Changed lines of the file:
@@
 AR Path="/5CD47361/5CD6BE5F/5CFD45EB" Ref="SW?"  Part="1"
 AR Path="/5CF23C1A/5CD6BE5F/5CFD45EB" Ref="SW?"  Part="1"
-AR Path="/5CF23C1A/5CFD2A64/5CFD45EB" Ref="SW?"  Part="1"
-F 0 "SW?" V 1200 2250 50  0000 L CNN
+AR Path="/5CF23C1A/5CFD2A64/5CFD45EB" Ref="SW3"  Part="1"
+F 0 "SW3" V 1200 2250 50  0000 L CNN
 F 1 "USER_BUTTON1" V 1250 2250 50  0000 L CNN
 F 2 "footprint-lib:SW_SPST_CK_RS282G05A3" H 1250 2300 50  0001 C CNN
@@
 AR Path="/5CD47361/5CD6BE5F/5CFD45F1" Ref="R?"  Part="1"
 AR Path="/5CF23C1A/5CD6BE5F/5CFD45F1" Ref="R?"  Part="1"
-AR Path="/5CF23C1A/5CFD2A64/5CFD45F1" Ref="R?"  Part="1"
-F 0 "R?" H 1350 1700 50  0000 L CNN
+AR Path="/5CF23C1A/5CFD2A64/5CFD45F1" Ref="R22"  Part="1"
+F 0 "R22" H 1350 1700 50  0000 L CNN
 F 1 "R471,0603" H 1350 1650 50  0000 L CNN
 F 2 "Resistor_SMD:R_0603_1608Metric_Pad1.05x0.95mm_HandSolder" H 1250 1650 50  0001 C CNN
@@
 AR Path="/5CD47361/5CD6BE5F/5CFD45FA" Ref="#PWR?"  Part="1"
 AR Path="/5CF23C1A/5CD6BE5F/5CFD45FA" Ref="#PWR?"  Part="1"
-AR Path="/5CF23C1A/5CFD2A64/5CFD45FA" Ref="#PWR?"  Part="1"
-F 0 "#PWR?" H 1250 2250 50  0001 C CNN
+AR Path="/5CF23C1A/5CFD2A64/5CFD45FA" Ref="#PWR056"  Part="1"
+F 0 "#PWR056" H 1250 2250 50  0001 C CNN
 F 1 "GND" H 1300 2300 50  0000 C CNN
 F 2 "" H 1250 2500 50  0001 C CNN
@@
 AR Path="/5CD47361/5CD6BE5F/5CFD4601" Ref="SW?"  Part="1"
 AR Path="/5CF23C1A/5CD6BE5F/5CFD4601" Ref="SW?"  Part="1"
-AR Path="/5CF23C1A/5CFD2A64/5CFD4601" Ref="SW?"  Part="1"
-F 0 "SW?" V 2150 2250 50  0000 L CNN
+AR Path="/5CF23C1A/5CFD2A64/5CFD4601" Ref="SW4"  Part="1"
+F 0 "SW4" V 2150 2250 50  0000 L CNN
 F 1 "USER_BUTTON2" V 2200 2250 50  0000 L CNN
 F 2 "footprint-lib:SW_SPST_CK_RS282G05A3" H 2200 2300 50  0001 C CNN
@@
 AR Path="/5CD47361/5CD6BE5F/5CFD4607" Ref="R?"  Part="1"
 AR Path="/5CF23C1A/5CD6BE5F/5CFD4607" Ref="R?"  Part="1"
-AR Path="/5CF23C1A/5CFD2A64/5CFD4607" Ref="R?"  Part="1"
-F 0 "R?" H 2300 1700 50  0000 L CNN
+AR Path="/5CF23C1A/5CFD2A64/5CFD4607" Ref="R23"  Part="1"
+F 0 "R23" H 2300 1700 50  0000 L CNN
 F 1 "R471,0603" H 2300 1650 50  0000 L CNN
 F 2 "Resistor_SMD:R_0603_1608Metric_Pad1.05x0.95mm_HandSolder" H 2200 1650 50  0001 C CNN
@@
 AR Path="/5CD47361/5CD6BE5F/5CFD4610" Ref="#PWR?"  Part="1"
 AR Path="/5CF23C1A/5CD6BE5F/5CFD4610" Ref="#PWR?"  Part="1"
-AR Path="/5CF23C1A/5CFD2A64/5CFD4610" Ref="#PWR?"  Part="1"
-F 0 "#PWR?" H 2200 2250 50  0001 C CNN
+AR Path="/5CF23C1A/5CFD2A64/5CFD4610" Ref="#PWR057"  Part="1"
+F 0 "#PWR057" H 2200 2250 50  0001 C CNN
 F 1 "GND" H 2250 2300 50  0000 C CNN
 F 2 "" H 2200 2500 50  0001 C CNN
@@
 AR Path="/5CD47361/5CD6BE5F/5CFD4619" Ref="SW?"  Part="1"
 AR Path="/5CF23C1A/5CD6BE5F/5CFD4619" Ref="SW?"  Part="1"
-AR Path="/5CF23C1A/5CFD2A64/5CFD4619" Ref="SW?"  Part="1"
-F 0 "SW?" V 3000 2250 50  0000 L CNN
+AR Path="/5CF23C1A/5CFD2A64/5CFD4619" Ref="SW5"  Part="1"
+F 0 "SW5" V 3000 2250 50  0000 L CNN
 F 1 "USER_BUTTON1" V 3050 2250 50  0000 L CNN
 F 2 "footprint-lib:SW_SPST_CK_RS282G05A3" H 3050 2300 50  0001 C CNN
@@
 AR Path="/5CD47361/5CD6BE5F/5CFD461F" Ref="R?"  Part="1"
 AR Path="/5CF23C1A/5CD6BE5F/5CFD461F" Ref="R?"  Part="1"
-AR Path="/5CF23C1A/5CFD2A64/5CFD461F" Ref="R?"  Part="1"
-F 0 "R?" H 3150 1700 50  0000 L CNN
+AR Path="/5CF23C1A/5CFD2A64/5CFD461F" Ref="R24"  Part="1"
+F 0 "R24" H 3150 1700 50  0000 L CNN
 F 1 "R471,0603" H 3150 1650 50  0000 L CNN
 F 2 "Resistor_SMD:R_0603_1608Metric_Pad1.05x0.95mm_HandSolder" H 3050 1650 50  0001 C CNN
@@
 AR Path="/5CD47361/5CD6BE5F/5CFD4628" Ref="#PWR?"  Part="1"
 AR Path="/5CF23C1A/5CD6BE5F/5CFD4628" Ref="#PWR?"  Part="1"
-AR Path="/5CF23C1A/5CFD2A64/5CFD4628" Ref="#PWR?"  Part="1"
-F 0 "#PWR?" H 3050 2250 50  0001 C CNN
+AR Path="/5CF23C1A/5CFD2A64/5CFD4628" Ref="#PWR058"  Part="1"
+F 0 "#PWR058" H 3050 2250 50  0001 C CNN
 F 1 "GND" H 3100 2300 50  0000 C CNN
 F 2 "" H 3050 2500 50  0001 C CNN
