File: hardware/user_button.sch (KiCad schematic (older format))
At the start: 8 parts

Commit message: after DRC,
Parts:
- gave numbers to parts that had none: 8
Changed lines of the file:
@@
 $EndDescr
 $Comp
-L taobao-components:EC11_VERTICAL SW?
+L taobao-components:EC11_VERTICAL SW6
 U 1 1 5CEC3ACC
 P 3900 2700
-F 0 "SW?" H 3900 2300 50  0000 C CNN
+F 0 "SW6" H 3900 2300 50  0000 C CNN
 F 1 "EC11_VERTICAL" H 3900 2400 50  0000 C CNN
 F 2 "footprint-lib:RotaryEncoder_Alps_EC11E_Vertical_H20mm" H 3900 2350 50  0001 C CNN
@@
 $EndBitmap
 $Comp
-L taobao-r:R273,0603 R?
+L taobao-r:R273,0603 R31
 U 1 1 5CED60AF
 P 3150 2300
-F 0 "R?" V 2900 2300 50  0000 C CNN
+F 0 "R31" V 2900 2300 50  0000 C CNN
 F 1 "R273,0603" V 3000 2300 50  0000 C CNN
 F 2 "Resistor_SMD:R_0603_1608Metric_Pad1.05x0.95mm_HandSolder" H 3150 2300 50  0001 C CNN
@@
 $EndComp
 $Comp
-L taobao-r:R273,0603 R?
+L taobao-r:R273,0603 R32
 U 1 1 5CED6622
 P 3150 2800
-F 0 "R?" V 2900 2800 50  0000 C CNN
+F 0 "R32" V 2900 2800 50  0000 C CNN
 F 1 "R273,0603" V 3000 2800 50  0000 C CNN
 F 2 "Resistor_SMD:R_0603_1608Metric_Pad1.05x0.95mm_HandSolder" H 3150 2800 50  0001 C CNN
@@
 $EndComp
 $Comp
-L taobao-r:R273,0603 R?
+L taobao-r:R273,0603 R33
 U 1 1 5CED67EF
 P 3150 3250
-F 0 "R?" V 2900 3250 50  0000 C CNN
+F 0 "R33" V 2900 3250 50  0000 C CNN
 F 1 "R273,0603" V 3000 3250 50  0000 C CNN
 F 2 "Resistor_SMD:R_0603_1608Metric_Pad1.05x0.95mm_HandSolder" H 3150 3250 50  0001 C CNN
@@
 $EndComp
 $Comp
-L taobao-c:C104,0603 C?
+L taobao-c:C104,0603 C15
 U 1 1 5CED6CD1
 P 2800 3450
-F 0 "C?" H 2900 3500 50  0000 L CNN
+F 0 "C15" H 2900 3500 50  0000 L CNN
 F 1 "C104,0603" H 2900 3450 50  0000 L CNN
 F 2 "Capacitor_SMD:C_0603_1608Metric_Pad1.05x0.95mm_HandSolder" H 2800 3450 50  0001 C CNN
@@
 $EndComp
 $Comp
-L taobao-c:C104,0603 C?
+L taobao-c:C104,0603 C14
 U 1 1 5CED7298
 P 2800 2950
-F 0 "C?" H 2900 3000 50  0000 L CNN
+F 0 "C14" H 2900 3000 50  0000 L CNN
 F 1 "C104,0603" H 2900 2950 50  0000 L CNN
 F 2 "Capacitor_SMD:C_0603_1608Metric_Pad1.05x0.95mm_HandSolder" H 2800 2950 50  0001 C CNN
@@
 $EndComp
 $Comp
-L taobao-c:C104,0603 C?
+L taobao-c:C104,0603 C13
 U 1 1 5CED75A5
 P 2800 2500
-F 0 "C?" H 2900 2550 50  0000 L CNN
+F 0 "C13" H 2900 2550 50  0000 L CNN
 F 1 "C104,0603" H 2900 2500 50  0000 L CNN
 F 2 "Capacitor_SMD:C_0603_1608Metric_Pad1.05x0.95mm_HandSolder" H 2800 2500 50  0001 C CNN
@@
 	2800 3250 2800 3350
 $Comp
-L power:GND #PWR?
+L power:GND #PWR068
 U 1 1 5CED86F3
 P 2800 2650
-F 0 "#PWR?" H 2800 2400 50  0001 C CNN
+F 0 "#PWR068" H 2800 2400 50  0001 C CNN
 F 1 "GND" H 2850 2450 50  0000 C CNN
 F 2 "" H 2800 2650 50  0001 C CNN
@@
 	2800 2650 2800 2600
 $Comp
-L power:GND #PWR?
+L power:GND #PWR070
 U 1 1 5CED8B04
 P 2800 3100
-F 0 "#PWR?" H 2800 2850 50  0001 C CNN
+F 0 "#PWR070" H 2800 2850 50  0001 C CNN
 F 1 "GND" H 2850 2900 50  0000 C CNN
 F 2 "" H 2800 3100 50  0001 C CNN
@@
 	2800 3100 2800 3050
 $Comp
-L power:GND #PWR?
+L power:GND #PWR071
 U 1 1 5CED8F95
 P 2800 3600
-F 0 "#PWR?" H 2800 3350 50  0001 C CNN
+F 0 "#PWR071" H 2800 3350 50  0001 C CNN
 F 1 "GND" H 2850 3400 50  0000 C CNN
 F 2 "" H 2800 3600 50  0001 C CNN
@@
 	2800 3600 2800 3550
 $Comp
-L power:GND #PWR?
+L power:GND #PWR067
 U 1 1 5CED947F
 P 3350 2600
-F 0 "#PWR?" H 3350 2350 50  0001 C CNN
+F 0 "#PWR067" H 3350 2350 50  0001 C CNN
 F 1 "GND" H 3400 2400 50  0000 C CNN
 F 2 "" H 3350 2600 50  0001 C CNN
@@
 $EndComp
 $Comp
-L power:GND #PWR?
+L power:GND #PWR069
 U 1 1 5CED96CA
 P 4400 2900
-F 0 "#PWR?" H 4400 2650 50  0001 C CNN
+F 0 "#PWR069" H 4400 2650 50  0001 C CNN
 F 1 "GND" H 4450 2700 50  0000 C CNN
 F 2 "" H 4400 2900 50  0001 C CNN
@@
 Connection ~ 2800 3250
 $Comp
-L Connector:Conn_01x03_Female J?
+L Connector:Conn_01x03_Female J10
 U 1 1 5CF225E9
 P 1100 2200
-F 0 "J?" H 950 2500 50  0000 C CNN
+F 0 "J10" H 950 2500 50  0000 C CNN
 F 1 "ROT_ENC_HEADER" H 950 2400 50  0000 C CNN
 F 2 "Connector_PinHeader_1.27mm:PinHeader_1x03_P1.27mm_Vertical" H 1100 2200 50  0001 C CNN
