File: hardware/GSM.sch (KiCad schematic (older format))
At the start: 4 parts

Commit message: after DRC,
Parts:
- gave numbers to parts that had none: 4
Connections:
- wire segments 13 -> 14
Changed lines of the file:
@@
 $Descr User 8500 5500
 encoding utf-8
-Sheet 11 15
+Sheet 10 15
 Title ""
 Date ""
@@
 $EndBitmap
 $Comp
-L Connector:Conn_01x04_Female J?
+L Connector:Conn_01x04_Female J7
 U 1 1 5CF6031E
 P 1050 2150
-AR Path="/5CF23C6C/5CF6031E" Ref="J?"  Part="1"
+AR Path="/5CF23C6C/5CF6031E" Ref="J7"  Part="1"
 AR Path="/5CF2E587/5CF6031E" Ref="J?"  Part="1"
-F 0 "J?" H 942 2435 50  0000 C CNN
+F 0 "J7" H 942 2435 50  0000 C CNN
 F 1 "TXD_HEADER" H 942 2344 50  0000 C CNN
 F 2 "" H 1050 2150 50  0001 C CNN
@@
 $EndComp
 $Comp
-L power:+3V3 #PWR?
+L power:+3V3 #PWR059
 U 1 1 5CF607EB
 P 1550 1450
-AR Path="/5CF23C6C/5CF607EB" Ref="#PWR?"  Part="1"
+AR Path="/5CF23C6C/5CF607EB" Ref="#PWR059"  Part="1"
 AR Path="/5CF2E587/5CF607EB" Ref="#PWR?"  Part="1"
-F 0 "#PWR?" H 1550 1300 50  0001 C CNN
+F 0 "#PWR059" H 1550 1300 50  0001 C CNN
 F 1 "+3V3" H 1565 1623 50  0000 C CNN
 F 2 "" H 1550 1450 50  0001 C CNN
@@
 $EndComp
 $Comp
-L power:GND #PWR?
+L power:GND #PWR060
 U 1 1 5CF60DB4
 P 1650 2600
-AR Path="/5CF23C6C/5CF60DB4" Ref="#PWR?"  Part="1"
+AR Path="/5CF23C6C/5CF60DB4" Ref="#PWR060"  Part="1"
 AR Path="/5CF2E587/5CF60DB4" Ref="#PWR?"  Part="1"
-F 0 "#PWR?" H 1650 2350 50  0001 C CNN
+F 0 "#PWR060" H 1650 2350 50  0001 C CNN
 F 1 "GND" H 1655 2427 50  0000 C CNN
 F 2 "" H 1650 2600 50  0001 C CNN
@@
 	1250 2250 1550 2250
 $Comp
-L my_solder_jumper:SolderJumper_2_Open_round JP?
+L my_solder_jumper:SolderJumper_2_Open_round JP8
 U 1 1 5CF62D5D
 P 1550 1700
-AR Path="/5CF23C6C/5CF62D5D" Ref="JP?"  Part="1"
+AR Path="/5CF23C6C/5CF62D5D" Ref="JP8"  Part="1"
 AR Path="/5CF2E587/5CF62D5D" Ref="JP?"  Part="1"
-F 0 "JP?" V 1504 1768 50  0000 L CNN
+F 0 "JP8" V 1504 1768 50  0000 L CNN
 F 1 "PWR_EN" V 1595 1768 50  0000 L CNN
 F 2 "Jumper:SolderJumper-2_P1.3mm_Open_RoundedPad1.0x1.5mm" H 1550 1700 50  0001 C CNN
@@
 	1250 2050 1550 2050
 Wire Wire Line
-	1550 2050 1550 1850
+	1550 2050 1550 1900
 Text Label 1100 750  2    50   ~ 0
 TXD
@@
 P 2300 2600
 AR Path="/5CF23B4E/5CFC0F9F" Ref="#PWR?"  Part="1"
-AR Path="/5CF23C6C/5CFC0F9F" Ref="#PWR?"  Part="1"
-F 0 "#PWR?" H 2300 2350 50  0001 C CNN
+AR Path="/5CF23C6C/5CFC0F9F" Ref="#PWR061"  Part="1"
+F 0 "#PWR061" H 2300 2350 50  0001 C CNN
 F 1 "GND" H 2350 2400 50  0000 C CNN
 F 2 "" H 2300 2600 50  0001 C CNN
@@
 P 2300 2200
 AR Path="/5CF23B4E/5CFC0FA7" Ref="R?"  Part="1"
-AR Path="/5CF23C6C/5CFC0FA7" Ref="R?"  Part="1"
-F 0 "R?" H 2359 2246 50  0000 L CNN
+AR Path="/5CF23C6C/5CFC0FA7" Ref="R25"  Part="1"
+F 0 "R25" H 2359 2246 50  0000 L CNN
 F 1 "R511,0603" H 2359 2155 50  0000 L CNN
 F 2 "Resistor_SMD:R_0603_1608Metric_Pad1.05x0.95mm_HandSolder" H 2300 2200 50  0001 C CNN
@@
 P 2300 2450
 AR Path="/5CF23B4E/5CFC0FAD" Ref="D?"  Part="1"
-AR Path="/5CF23C6C/5CFC0FAD" Ref="D?"  Part="1"
-F 0 "D?" V 2346 2382 50  0000 R CNN
+AR Path="/5CF23C6C/5CFC0FAD" Ref="D6"  Part="1"
+F 0 "D6" V 2346 2382 50  0000 R CNN
 F 1 "LED_GREEN,0603" V 2255 2382 50  0000 R CNN
 F 2 "footprint-lib:LED_0603_1608Metric" V 2300 2450 50  0001 C CNN
@@
 Wire Wire Line
 	2300 1900 2300 2100
+Connection ~ 1550 1900
+Wire Wire Line
+	1550 1900 1550 1850
 $EndSCHEMATC

Commit message: after routing,
Parts:
- J7: value TXD_HEADER -> GSM_TX_HEADER; footprint (none) -> Connector_PinHeader_2.54mm:PinHeader_1x04_P2.54mm_Vertical
Changed lines of the file:
@@
 AR Path="/5CF2E587/5CF6031E" Ref="J?"  Part="1"
 F 0 "J7" H 942 2435 50  0000 C CNN
-F 1 "TXD_HEADER" H 942 2344 50  0000 C CNN
-F 2 "" H 1050 2150 50  0001 C CNN
+F 1 "GSM_TX_HEADER" H 942 2344 50  0000 C CNN
+F 2 "Connector_PinHeader_2.54mm:PinHeader_1x04_P2.54mm_Vertical" H 1050 2150 50  0001 C CNN
 F 3 "~" H 1050 2150 50  0001 C CNN
 	1    1050 2150
