File: hardware/humidity_sensor.sch (KiCad schematic (older format))
At the start: 8 parts

Commit message: after DRC,
Parts:
- gave numbers to parts that had none: 8
Connections:
- wire segments 29 -> 30
Changed lines of the file:
@@
 $EndBitmap
 $Comp
-L taobao-components:SHT20 U?
+L taobao-components:SHT20 U2
 U 1 1 5CF2A99C
 P 2400 3200
-F 0 "U?" V 2446 3427 50  0000 L CNN
+F 0 "U2" V 2446 3427 50  0000 L CNN
 F 1 "SHT20" V 2355 3427 50  0000 L CNN
 F 2 "footprint-lib:SHT20" H 2400 3200 50  0001 C CNN
@@
 $EndComp
 $Comp
-L taobao-components:I2C_HEADER,2.54 J?
+L taobao-components:I2C_HEADER,2.54 J2
 U 1 1 5CF2D2E3
 P 1000 3300
-F 0 "J?" H 972 3232 50  0000 R CNN
+F 0 "J2" H 972 3232 50  0000 R CNN
 F 1 "I2C_HEADER,2.54" H 972 3323 50  0000 R CNN
 F 2 "Connector_PinHeader_2.54mm:PinHeader_1x02_P2.54mm_Vertical" H 1000 2900 50  0001 C CNN
@@
 $EndComp
 $Comp
-L power:+3V3 #PWR?
+L power:+3V3 #PWR010
 U 1 1 5CF2D9F9
 P 2400 2200
-F 0 "#PWR?" H 2400 2050 50  0001 C CNN
+F 0 "#PWR010" H 2400 2050 50  0001 C CNN
 F 1 "+3V3" H 2415 2373 50  0000 C CNN
 F 2 "" H 2400 2200 50  0001 C CNN
@@
 $EndComp
 $Comp
-L power:GND #PWR?
+L power:GND #PWR014
 U 1 1 5CF2DE3B
 P 2400 4100
-F 0 "#PWR?" H 2400 3850 50  0001 C CNN
+F 0 "#PWR014" H 2400 3850 50  0001 C CNN
 F 1 "GND" H 2405 3927 50  0000 C CNN
 F 2 "" H 2400 4100 50  0001 C CNN
@@
 	2400 3650 2400 4100
 $Comp
-L power:GND #PWR?
+L power:GND #PWR011
 U 1 1 5CF2EA48
 P 2900 3400
-F 0 "#PWR?" H 2900 3150 50  0001 C CNN
+F 0 "#PWR011" H 2900 3150 50  0001 C CNN
 F 1 "GND" H 2905 3227 50  0000 C CNN
 F 2 "" H 2900 3400 50  0001 C CNN
@@
 	2900 3200 2900 3400
 $Comp
-L power:+3V3 #PWR?
+L power:+3V3 #PWR013
 U 1 1 5CF2EF97
 P 1100 3850
-F 0 "#PWR?" H 1100 3700 50  0001 C CNN
+F 0 "#PWR013" H 1100 3700 50  0001 C CNN
 F 1 "+3V3" H 1115 4023 50  0000 C CNN
 F 2 "" H 1100 3850 50  0001 C CNN
@@
 $EndComp
 $Comp
-L power:GND #PWR?
+L power:GND #PWR015
 U 1 1 5CF2F1C5
 P 1100 4350
-F 0 "#PWR?" H 1100 4100 50  0001 C CNN
+F 0 "#PWR015" H 1100 4100 50  0001 C CNN
 F 1 "GND" H 1105 4177 50  0000 C CNN
 F 2 "" H 1100 4350 50  0001 C CNN
@@
 $EndComp
 $Comp
-L taobao-c:C106,0603 C?
+L taobao-c:C106,0603 C2
 U 1 1 5CF2F5B3
 P 1100 4100
-F 0 "C?" H 1192 4146 50  0000 L CNN
+F 0 "C2" H 1192 4146 50  0000 L CNN
 F 1 "C106,0603" H 1192 4055 50  0000 L CNN
 F 2 "Capacitor_SMD:C_0603_1608Metric_Pad1.05x0.95mm_HandSolder" H 1100 4100 50  0001 C CNN
@@
 AR Path="/5CF23C1A/5CF86AD5" Ref="#PWR?"  Part="1"
 AR Path="/5CF23B0A/5CF86AD5" Ref="#PWR?"  Part="1"
-AR Path="/5CF23B1B/5CF86AD5" Ref="#PWR?"  Part="1"
-F 0 "#PWR?" H 1950 1050 50  0001 C CNN
+AR Path="/5CF23B1B/5CF86AD5" Ref="#PWR09"  Part="1"
+F 0 "#PWR09" H 1950 1050 50  0001 C CNN
 F 1 "+3V3" H 1950 1400 50  0000 C CNN
 F 2 "" H 1950 1200 50  0001 C CNN
@@
 P 1400 1200
 AR Path="/5CF23B0A/5CF86ADB" Ref="R?"  Part="1"
-AR Path="/5CF23B1B/5CF86ADB" Ref="R?"  Part="1"
-F 0 "R?" V 1204 1200 50  0000 C CNN
+AR Path="/5CF23B1B/5CF86ADB" Ref="R4"  Part="1"
+F 0 "R4" V 1204 1200 50  0000 C CNN
 F 1 "R473,0603" V 1295 1200 50  0000 C CNN
 F 2 "Resistor_SMD:R_0603_1608Metric_Pad1.05x0.95mm_HandSolder" H 1400 1200 50  0001 C CNN
@@
 P 1400 1300
 AR Path="/5CF23B0A/5CF86AE1" Ref="R?"  Part="1"
-AR Path="/5CF23B1B/5CF86AE1" Ref="R?"  Part="1"
-F 0 "R?" V 1504 1300 50  0000 C CNN
+AR Path="/5CF23B1B/5CF86AE1" Ref="R5"  Part="1"
+F 0 "R5" V 1504 1300 50  0000 C CNN
 F 1 "R473,0603" V 1595 1300 50  0000 C CNN
 F 2 "Resistor_SMD:R_0603_1608Metric_Pad1.05x0.95mm_HandSolder" H 1400 1300 50  0001 C CNN
@@
 	1850 1250 1850 1300
 $Comp
-L my_solder_jumper:SolderJumper_2_Open_round JP?
+L my_solder_jumper:SolderJumper_2_Open_round JP2
 U 1 1 5CF8C196
 P 2400 2500
-F 0 "JP?" V 2354 2568 50  0000 L CNN
+F 0 "JP2" V 2354 2568 50  0000 L CNN
 F 1 "SHT20_EN" V 2445 2568 50  0000 L CNN
 F 2 "Jumper:SolderJumper-2_P1.3mm_Open_RoundedPad1.0x1.5mm" H 2400 2500 50  0001 C CNN
@@
 $EndComp
 Wire Wire Line
-	2400 2650 2400 2750
+	2400 2650 2400 2700
 Wire Wire Line
 	2400 2200 2400 2350
@@
 P 3150 3400
 AR Path="/5CF23B4E/5CFBF5F9" Ref="#PWR?"  Part="1"
-AR Path="/5CF23B1B/5CFBF5F9" Ref="#PWR?"  Part="1"
-F 0 "#PWR?" H 3150 3150 50  0001 C CNN
+AR Path="/5CF23B1B/5CFBF5F9" Ref="#PWR012"  Part="1"
+F 0 "#PWR012" H 3150 3150 50  0001 C CNN
 F 1 "GND" H 3200 3200 50  0000 C CNN
 F 2 "" H 3150 3400 50  0001 C CNN
@@
 P 3150 3000
 AR Path="/5CF23B4E/5CFBF601" Ref="R?"  Part="1"
-AR Path="/5CF23B1B/5CFBF601" Ref="R?"  Part="1"
-F 0 "R?" H 3209 3046 50  0000 L CNN
+AR Path="/5CF23B1B/5CFBF601" Ref="R6"  Part="1"
+F 0 "R6" H 3209 3046 50  0000 L CNN
 F 1 "R511,0603" H 3209 2955 50  0000 L CNN
 F 2 "Resistor_SMD:R_0603_1608Metric_Pad1.05x0.95mm_HandSolder" H 3150 3000 50  0001 C CNN
@@
 P 3150 3250
 AR Path="/5CF23B4E/5CFBF607" Ref="D?"  Part="1"
-AR Path="/5CF23B1B/5CFBF607" Ref="D?"  Part="1"
-F 0 "D?" V 3196 3182 50  0000 R CNN
+AR Path="/5CF23B1B/5CFBF607" Ref="D2"  Part="1"
+F 0 "D2" V 3196 3182 50  0000 R CNN
 F 1 "LED_GREEN,0603" V 3105 3182 50  0000 R CNN
 F 2 "footprint-lib:LED_0603_1608Metric" V 3150 3250 50  0001 C CNN
@@
 Wire Wire Line
 	3150 2700 3150 2900
+Connection ~ 2400 2700
+Wire Wire Line
+	2400 2700 2400 2750
 $EndSCHEMATC

Commit message: after routing,
Parts:
- J2: footprint Connector_PinHeader_2.54mm:PinHeader_1x02_P2.54mm_Vertical -> footprint-lib:I2C_DEBUG,2.54
Changed lines of the file:
@@
 F 0 "J2" H 972 3232 50  0000 R CNN
 F 1 "I2C_HEADER,2.54" H 972 3323 50  0000 R CNN
-F 2 "Connector_PinHeader_2.54mm:PinHeader_1x02_P2.54mm_Vertical" H 1000 2900 50  0001 C CNN
+F 2 "footprint-lib:I2C_DEBUG,2.54" H 1000 2900 50  0001 C CNN
 F 3 "" H 1000 3250 50  0001 C CNN
 	1    1000 3300
