File: hardware/i2c_input.sch (KiCad schematic (older format))
At the start: 3 parts

Commit message: after DRC,
Parts:
- gave numbers to parts that had none: 3
Changed lines of the file:
@@
 P 1250 4050
 AR Path="/5CF23B1B/5CF34BF5" Ref="J?"  Part="1"
-AR Path="/5CF23B71/5CF34BF5" Ref="J?"  Part="1"
-F 0 "J?" H 1222 3982 50  0000 R CNN
+AR Path="/5CF23B71/5CF34BF5" Ref="J11"  Part="1"
+F 0 "J11" H 1222 3982 50  0000 R CNN
 F 1 "I2C_HEADER,2.54" H 1222 4073 50  0000 R CNN
 F 2 "Connector_PinHeader_2.54mm:PinHeader_1x02_P2.54mm_Vertical" H 1250 3650 50  0001 C CNN
@@
 AR Path="/5CF23B0A/5CFC8CBF" Ref="#PWR?"  Part="1"
 AR Path="/5CF23B1B/5CFC8CBF" Ref="#PWR?"  Part="1"
-AR Path="/5CF23B71/5CFC8CBF" Ref="#PWR?"  Part="1"
-F 0 "#PWR?" H 1800 1100 50  0001 C CNN
+AR Path="/5CF23B71/5CFC8CBF" Ref="#PWR072"  Part="1"
+F 0 "#PWR072" H 1800 1100 50  0001 C CNN
 F 1 "+3V3" H 1800 1450 50  0000 C CNN
 F 2 "" H 1800 1250 50  0001 C CNN
@@
 AR Path="/5CF23B0A/5CFC8CC5" Ref="R?"  Part="1"
 AR Path="/5CF23B1B/5CFC8CC5" Ref="R?"  Part="1"
-AR Path="/5CF23B71/5CFC8CC5" Ref="R?"  Part="1"
-F 0 "R?" V 1054 1250 50  0000 C CNN
+AR Path="/5CF23B71/5CFC8CC5" Ref="R34"  Part="1"
+F 0 "R34" V 1054 1250 50  0000 C CNN
 F 1 "R473,0603" V 1145 1250 50  0000 C CNN
 F 2 "Resistor_SMD:R_0603_1608Metric_Pad1.05x0.95mm_HandSolder" H 1250 1250 50  0001 C CNN
@@
 AR Path="/5CF23B0A/5CFC8CCB" Ref="R?"  Part="1"
 AR Path="/5CF23B1B/5CFC8CCB" Ref="R?"  Part="1"
-AR Path="/5CF23B71/5CFC8CCB" Ref="R?"  Part="1"
-F 0 "R?" V 1354 1350 50  0000 C CNN
+AR Path="/5CF23B71/5CFC8CCB" Ref="R35"  Part="1"
+F 0 "R35" V 1354 1350 50  0000 C CNN
 F 1 "R473,0603" V 1445 1350 50  0000 C CNN
 F 2 "Resistor_SMD:R_0603_1608Metric_Pad1.05x0.95mm_HandSolder" H 1250 1350 50  0001 C CNN

Commit message: after routing,
Parts:
- J11: footprint Connector_PinHeader_2.54mm:PinHeader_1x02_P2.54mm_Vertical -> footprint-lib:I2C_DEBUG,2.54
Changed lines of the file:
@@
 F 0 "J11" H 1222 3982 50  0000 R CNN
 F 1 "I2C_HEADER,2.54" H 1222 4073 50  0000 R CNN
-F 2 "Connector_PinHeader_2.54mm:PinHeader_1x02_P2.54mm_Vertical" H 1250 3650 50  0001 C CNN
+F 2 "footprint-lib:I2C_DEBUG,2.54" H 1250 3650 50  0001 C CNN
 F 3 "" H 1250 4000 50  0001 C CNN
 	1    1250 4050
