File: hardware/i2c_output.sch (KiCad schematic (older format))
At the start: 3 parts

Commit message: after DRC,
Parts:
- gave numbers to parts that had none: 3
Changed lines of the file:
@@
 AR Path="/5CF23B71/5D001693" Ref="J?"  Part="1"
 AR Path="/5CF23D41/5D001693" Ref="J?"  Part="1"
-AR Path="/5CF23D02/5D001693" Ref="J?"  Part="1"
-F 0 "J?" H 672 882 50  0000 R CNN
+AR Path="/5CF23D02/5D001693" Ref="J8"  Part="1"
+F 0 "J8" H 672 882 50  0000 R CNN
 F 1 "I2C_HEADER,2.54" H 672 973 50  0000 R CNN
 F 2 "Connector_PinHeader_2.54mm:PinHeader_1x02_P2.54mm_Vertical" H 700 550 50  0001 C CNN
@@
 AR Path="/5CF23B1B/5D0016A0" Ref="#PWR?"  Part="1"
 AR Path="/5CF23D41/5D0016A0" Ref="#PWR?"  Part="1"
-AR Path="/5CF23D02/5D0016A0" Ref="#PWR?"  Part="1"
-F 0 "#PWR?" H 1750 1150 50  0001 C CNN
+AR Path="/5CF23D02/5D0016A0" Ref="#PWR062"  Part="1"
+F 0 "#PWR062" H 1750 1150 50  0001 C CNN
 F 1 "+3V3" H 1750 1500 50  0000 C CNN
 F 2 "" H 1750 1300 50  0001 C CNN
@@
 AR Path="/5CF23B1B/5D0016A6" Ref="R?"  Part="1"
 AR Path="/5CF23D41/5D0016A6" Ref="R?"  Part="1"
-AR Path="/5CF23D02/5D0016A6" Ref="R?"  Part="1"
-F 0 "R?" V 1004 1300 50  0000 C CNN
+AR Path="/5CF23D02/5D0016A6" Ref="R26"  Part="1"
+F 0 "R26" V 1004 1300 50  0000 C CNN
 F 1 "R473,0603" V 1095 1300 50  0000 C CNN
 F 2 "Resistor_SMD:R_0603_1608Metric_Pad1.05x0.95mm_HandSolder" H 1200 1300 50  0001 C CNN
@@
 AR Path="/5CF23B1B/5D0016AC" Ref="R?"  Part="1"
 AR Path="/5CF23D41/5D0016AC" Ref="R?"  Part="1"
-AR Path="/5CF23D02/5D0016AC" Ref="R?"  Part="1"
-F 0 "R?" V 1304 1400 50  0000 C CNN
+AR Path="/5CF23D02/5D0016AC" Ref="R27"  Part="1"
+F 0 "R27" V 1304 1400 50  0000 C CNN
 F 1 "R473,0603" V 1395 1400 50  0000 C CNN
 F 2 "Resistor_SMD:R_0603_1608Metric_Pad1.05x0.95mm_HandSolder" H 1200 1400 50  0001 C CNN

Commit message: after routing,
Parts:
- J8: footprint Connector_PinHeader_2.54mm:PinHeader_1x02_P2.54mm_Vertical -> footprint-lib:I2C_DEBUG,2.54
Changed lines of the file:
@@
 F 0 "J8" H 672 882 50  0000 R CNN
 F 1 "I2C_HEADER,2.54" H 672 973 50  0000 R CNN
-F 2 "Connector_PinHeader_2.54mm:PinHeader_1x02_P2.54mm_Vertical" H 700 550 50  0001 C CNN
+F 2 "footprint-lib:I2C_DEBUG,2.54" H 700 550 50  0001 C CNN
 F 3 "" H 700 900 50  0001 C CNN
 	1    700  950
