File: hardware/lcd.sch (KiCad schematic (older format))
At the start: 7 parts

Commit message: after DRC,
Parts:
- gave numbers to parts that had none: 7
Changed lines of the file:
@@
 AR Path="/5CF23B1B/5CF6EF09" Ref="J?"  Part="1"
 AR Path="/5CF23B71/5CF6EF09" Ref="J?"  Part="1"
-AR Path="/5CF23D41/5CF6EF09" Ref="J?"  Part="1"
-F 0 "J?" H 622 932 50  0000 R CNN
+AR Path="/5CF23D41/5CF6EF09" Ref="J9"  Part="1"
+F 0 "J9" H 622 932 50  0000 R CNN
 F 1 "I2C_HEADER,2.54" H 622 1023 50  0000 R CNN
 F 2 "Connector_PinHeader_2.54mm:PinHeader_1x02_P2.54mm_Vertical" H 650 600 50  0001 C CNN
@@
 	850  1050 1350 1050
 $Comp
-L taobao-board:SSD1306-OLED-I2C U?
+L taobao-board:SSD1306-OLED-I2C U8
 U 1 1 5CF6F58B
 P 2300 2800
-F 0 "U?" H 2778 2846 50  0000 L CNN
+F 0 "U8" H 2778 2846 50  0000 L CNN
 F 1 "SSD1306-OLED-I2C" H 2778 2755 50  0000 L CNN
 F 2 "" H 2300 2650 50  0001 C CNN
@@
 $EndComp
 $Comp
-L power:+3V3 #PWR?
+L power:+3V3 #PWR064
 U 1 1 5CF6F97A
 P 2700 1950
-F 0 "#PWR?" H 2700 1800 50  0001 C CNN
+F 0 "#PWR064" H 2700 1800 50  0001 C CNN
 F 1 "+3V3" H 2715 2123 50  0000 C CNN
 F 2 "" H 2700 1950 50  0001 C CNN
@@
 	2700 2650 2500 2650
 $Comp
-L power:GND #PWR?
+L power:GND #PWR065
 U 1 1 5CF6FD98
 P 3400 2900
-F 0 "#PWR?" H 3400 2650 50  0001 C CNN
+F 0 "#PWR065" H 3400 2650 50  0001 C CNN
 F 1 "GND" H 3405 2727 50  0000 C CNN
 F 2 "" H 3400 2900 50  0001 C CNN
@@
 P 3600 3300
 AR Path="/5CF23B4E/5CFC224F" Ref="#PWR?"  Part="1"
-AR Path="/5CF23D41/5CFC224F" Ref="#PWR?"  Part="1"
-F 0 "#PWR?" H 3600 3050 50  0001 C CNN
+AR Path="/5CF23D41/5CFC224F" Ref="#PWR066"  Part="1"
+F 0 "#PWR066" H 3600 3050 50  0001 C CNN
 F 1 "GND" H 3650 3100 50  0000 C CNN
 F 2 "" H 3600 3300 50  0001 C CNN
@@
 P 3600 2900
 AR Path="/5CF23B4E/5CFC2257" Ref="R?"  Part="1"
-AR Path="/5CF23D41/5CFC2257" Ref="R?"  Part="1"
-F 0 "R?" H 3659 2946 50  0000 L CNN
+AR Path="/5CF23D41/5CFC2257" Ref="R30"  Part="1"
+F 0 "R30" H 3659 2946 50  0000 L CNN
 F 1 "R511,0603" H 3659 2855 50  0000 L CNN
 F 2 "Resistor_SMD:R_0603_1608Metric_Pad1.05x0.95mm_HandSolder" H 3600 2900 50  0001 C CNN
@@
 P 3600 3150
 AR Path="/5CF23B4E/5CFC225D" Ref="D?"  Part="1"
-AR Path="/5CF23D41/5CFC225D" Ref="D?"  Part="1"
-F 0 "D?" V 3646 3082 50  0000 R CNN
+AR Path="/5CF23D41/5CFC225D" Ref="D7"  Part="1"
+F 0 "D7" V 3646 3082 50  0000 R CNN
 F 1 "LED_GREEN,0603" V 3555 3082 50  0000 R CNN
 F 2 "footprint-lib:LED_0603_1608Metric" V 3600 3150 50  0001 C CNN
@@
 	3600 2600 3600 2800
 $Comp
-L my_solder_jumper:SolderJumper_2_Open_round JP?
+L my_solder_jumper:SolderJumper_2_Open_round JP9
 U 1 1 5CFC36A6
 P 2700 2200
-F 0 "JP?" V 2654 2268 50  0000 L CNN
+F 0 "JP9" V 2654 2268 50  0000 L CNN
 F 1 "SolderJumper_2_Open_round" V 2745 2268 50  0000 L CNN
 F 2 "Jumper:SolderJumper-2_P1.3mm_Open_RoundedPad1.0x1.5mm" H 2700 2200 50  0001 C CNN
@@
 AR Path="/5CF23B0A/5CFE8B20" Ref="#PWR?"  Part="1"
 AR Path="/5CF23B1B/5CFE8B20" Ref="#PWR?"  Part="1"
-AR Path="/5CF23D41/5CFE8B20" Ref="#PWR?"  Part="1"
-F 0 "#PWR?" H 1700 1200 50  0001 C CNN
+AR Path="/5CF23D41/5CFE8B20" Ref="#PWR063"  Part="1"
+F 0 "#PWR063" H 1700 1200 50  0001 C CNN
 F 1 "+3V3" H 1700 1550 50  0000 C CNN
 F 2 "" H 1700 1350 50  0001 C CNN
@@
 AR Path="/5CF23B0A/5CFE8B26" Ref="R?"  Part="1"
 AR Path="/5CF23B1B/5CFE8B26" Ref="R?"  Part="1"
-AR Path="/5CF23D41/5CFE8B26" Ref="R?"  Part="1"
-F 0 "R?" V 954 1350 50  0000 C CNN
+AR Path="/5CF23D41/5CFE8B26" Ref="R28"  Part="1"
+F 0 "R28" V 954 1350 50  0000 C CNN
 F 1 "R473,0603" V 1045 1350 50  0000 C CNN
 F 2 "Resistor_SMD:R_0603_1608Metric_Pad1.05x0.95mm_HandSolder" H 1150 1350 50  0001 C CNN
@@
 AR Path="/5CF23B0A/5CFE8B2C" Ref="R?"  Part="1"
 AR Path="/5CF23B1B/5CFE8B2C" Ref="R?"  Part="1"
-AR Path="/5CF23D41/5CFE8B2C" Ref="R?"  Part="1"
-F 0 "R?" V 1254 1450 50  0000 C CNN
+AR Path="/5CF23D41/5CFE8B2C" Ref="R29"  Part="1"
+F 0 "R29" V 1254 1450 50  0000 C CNN
 F 1 "R473,0603" V 1345 1450 50  0000 C CNN
 F 2 "Resistor_SMD:R_0603_1608Metric_Pad1.05x0.95mm_HandSolder" H 1150 1450 50  0001 C CNN

Commit message: after routing,
Parts:
- J9: footprint Connector_PinHeader_2.54mm:PinHeader_1x02_P2.54mm_Vertical -> footprint-lib:I2C_DEBUG,2.54
- U8: footprint (none) -> footprint-lib:OLED_096_12864_SSD1306
Changed lines of the file:
@@
 F 0 "J9" H 622 932 50  0000 R CNN
 F 1 "I2C_HEADER,2.54" H 622 1023 50  0000 R CNN
-F 2 "Connector_PinHeader_2.54mm:PinHeader_1x02_P2.54mm_Vertical" H 650 600 50  0001 C CNN
+F 2 "footprint-lib:I2C_DEBUG,2.54" H 650 600 50  0001 C CNN
 F 3 "" H 650 950 50  0001 C CNN
 	1    650  1000
@@
 F 0 "U8" H 2778 2846 50  0000 L CNN
 F 1 "SSD1306-OLED-I2C" H 2778 2755 50  0000 L CNN
-F 2 "" H 2300 2650 50  0001 C CNN
+F 2 "footprint-lib:OLED_096_12864_SSD1306" H 2300 2650 50  0001 C CNN
 F 3 "" H 2300 2650 50  0001 C CNN
 	1    2300 2800
