File: hardware/power.sch (KiCad schematic (older format))
At the start: 0 parts

Commit message: after routing,
Parts:
- added C7: CP10uf,16V, Capacitor_SMD:CP_Elec_4x5.3, symbol taobao-cp:CP10uf,16V
- added C8: C106,0603, Capacitor_SMD:C_0603_1608Metric_Pad1.05x0.95mm_HandSolder, symbol taobao-c:C106,0603
- added J12, J13: 5V_header, Connector_PinHeader_2.54mm:PinHeader_1x02_P2.54mm_Vertical, symbol Connector:Conn_01x02_Female
- added U5: AMS1117-3.3, footprint-lib:AMS1117_SOT-223, symbol taobao-components:AMS1117-3.3
Connections:
- new net +3V3: C8.1, J13.2 (Pin_2), U5.2 (VO)
- new net +5V: C7.1, J12.2 (Pin_2), U5.3 (VI)
- new net GND: C7.2, C8.2, J12.1 (Pin_1), J13.1 (Pin_1), U5.1 (GND)
