File: hardware/WS2812.sch (KiCad schematic (older format))
At the start: 7 parts

Commit message: after DRC,
Parts:
- gave numbers to parts that had none: 7
Connections:
- no-connect marks 0 -> 1
Changed lines of the file:
@@
 $EndDescr
 $Comp
-L 74xGxx:74AHCT1G125 U?
+L 74xGxx:74AHCT1G125 U9
 U 1 1 5CFAEDA6
 P 1600 2500
-F 0 "U?" H 1600 2250 50  0001 C CNN
+F 0 "U9" H 1600 2250 50  0001 C CNN
 F 1 "74AHCT1G125" H 1600 2300 50  0000 C CNN
 F 2 "Package_TO_SOT_SMD:SOT-23-5_HandSoldering" H 1600 2500 50  0001 C CNN
@@
 $EndComp
 $Comp
-L taobao-c:C106,0805 C?
+L taobao-c:C106,0805 C16
 U 1 1 5CE4C478
 P 2700 1900
-F 0 "C?" V 2450 1900 50  0000 C CNN
+F 0 "C16" V 2450 1900 50  0000 C CNN
 F 1 "C106,0805" V 2550 1900 50  0000 C CNN
 F 2 "Capacitor_SMD:C_0805_2012Metric_Pad1.15x1.40mm_HandSolder" H 2700 1900 50  0001 C CNN
@@
 $EndComp
 $Comp
-L power:+5V #PWR?
+L power:+5V #PWR073
 U 1 1 5CF66BC4
 P 2400 1900
-F 0 "#PWR?" H 2400 1750 50  0001 C CNN
+F 0 "#PWR073" H 2400 1750 50  0001 C CNN
 F 1 "+5V" H 2450 2100 50  0000 C CNN
 F 2 "" H 2400 1900 50  0001 C CNN
@@
 $EndComp
 $Comp
-L power:GND #PWR?
+L power:GND #PWR074
 U 1 1 5CF671F3
 P 2850 1900
-F 0 "#PWR?" H 2850 1650 50  0001 C CNN
+F 0 "#PWR074" H 2850 1650 50  0001 C CNN
 F 1 "GND" V 2900 1750 50  0000 R CNN
 F 2 "" H 2850 1900 50  0001 C CNN
@@
 	1850 2500 2250 2500
 $Comp
-L power:GND #PWR?
+L power:GND #PWR082
 U 1 1 5CF6D6CD
 P 2550 2950
-F 0 "#PWR?" H 2550 2700 50  0001 C CNN
+F 0 "#PWR082" H 2550 2700 50  0001 C CNN
 F 1 "GND" H 2600 2750 50  0000 C CNN
 F 2 "" H 2550 2950 50  0001 C CNN
@@
 	2550 2800 2550 2950
 $Comp
-L taobao-c:C106,0805 C?
+L taobao-c:C106,0805 C17
 U 1 1 5CF6DBC3
 P 3700 1900
-F 0 "C?" V 3450 1900 50  0000 C CNN
+F 0 "C17" V 3450 1900 50  0000 C CNN
 F 1 "C106,0805" V 3550 1900 50  0000 C CNN
 F 2 "Capacitor_SMD:C_0805_2012Metric_Pad1.15x1.40mm_HandSolder" H 3700 1900 50  0001 C CNN
@@
 $EndComp
 $Comp
-L power:+5V #PWR?
+L power:+5V #PWR075
 U 1 1 5CF6DBCD
 P 3350 1900
-F 0 "#PWR?" H 3350 1750 50  0001 C CNN
+F 0 "#PWR075" H 3350 1750 50  0001 C CNN
 F 1 "+5V" H 3400 2100 50  0000 C CNN
 F 2 "" H 3350 1900 50  0001 C CNN
@@
 $EndComp
 $Comp
-L power:GND #PWR?
+L power:GND #PWR076
 U 1 1 5CF6DBD7
 P 3850 1900
-F 0 "#PWR?" H 3850 1650 50  0001 C CNN
+F 0 "#PWR076" H 3850 1650 50  0001 C CNN
 F 1 "GND" V 3900 1750 50  0000 R CNN
 F 2 "" H 3850 1900 50  0001 C CNN
@@
 	2850 2500 3250 2500
 $Comp
-L taobao-c:C106,0805 C?
+L taobao-c:C106,0805 C18
 U 1 1 5CF6F5B1
 P 4700 1900
-F 0 "C?" V 4450 1900 50  0000 C CNN
+F 0 "C18" V 4450 1900 50  0000 C CNN
 F 1 "C106,0805" V 4550 1900 50  0000 C CNN
 F 2 "Capacitor_SMD:C_0805_2012Metric_Pad1.15x1.40mm_HandSolder" H 4700 1900 50  0001 C CNN
@@
 $EndComp
 $Comp
-L power:+5V #PWR?
+L power:+5V #PWR077
 U 1 1 5CF6F5BB
 P 4300 1900
-F 0 "#PWR?" H 4300 1750 50  0001 C CNN
+F 0 "#PWR077" H 4300 1750 50  0001 C CNN
 F 1 "+5V" H 4350 2100 50  0000 C CNN
 F 2 "" H 4300 1900 50  0001 C CNN
@@
 $EndComp
 $Comp
-L power:GND #PWR?
+L power:GND #PWR078
 U 1 1 5CF6F5C5
 P 4850 1900
-F 0 "#PWR?" H 4850 1650 50  0001 C CNN
+F 0 "#PWR078" H 4850 1650 50  0001 C CNN
 F 1 "GND" V 4900 1750 50  0000 R CNN
 F 2 "" H 4850 1900 50  0001 C CNN
@@
 	4550 1900 4600 1900
 $Comp
-L power:GND #PWR?
+L power:GND #PWR083
 U 1 1 5CF76439
 P 3550 2950
-F 0 "#PWR?" H 3550 2700 50  0001 C CNN
+F 0 "#PWR083" H 3550 2700 50  0001 C CNN
 F 1 "GND" H 3600 2750 50  0000 C CNN
 F 2 "" H 3550 2950 50  0001 C CNN
@@
 	3550 2800 3550 2950
 $Comp
-L power:GND #PWR?
+L power:GND #PWR084
 U 1 1 5CF780F7
 P 4550 2950
-F 0 "#PWR?" H 4550 2700 50  0001 C CNN
+F 0 "#PWR084" H 4550 2700 50  0001 C CNN
 F 1 "GND" H 4600 2750 50  0000 C CNN
 F 2 "" H 4550 2950 50  0001 C CNN
@@
 	4550 2800 4550 2950
 $Comp
-L power:+5V #PWR?
+L power:+5V #PWR079
 U 1 1 5CEC2C6D
 P 1650 2200
-F 0 "#PWR?" H 1650 2050 50  0001 C CNN
+F 0 "#PWR079" H 1650 2050 50  0001 C CNN
 F 1 "+5V" H 1700 2400 50  0000 C CNN
 F 2 "" H 1650 2200 50  0001 C CNN
@@
 $EndComp
 $Comp
-L power:GND #PWR?
+L power:GND #PWR081
 U 1 1 5CEC323C
 P 1650 2800
-F 0 "#PWR?" H 1650 2550 50  0001 C CNN
+F 0 "#PWR081" H 1650 2550 50  0001 C CNN
 F 1 "GND" H 1700 2600 50  0000 C CNN
 F 2 "" H 1650 2800 50  0001 C CNN
@@
 	1650 2200 1650 2450
 $Comp
-L power:GND #PWR?
+L power:GND #PWR080
 U 1 1 5CEC5733
 P 1500 2250
-F 0 "#PWR?" H 1500 2000 50  0001 C CNN
+F 0 "#PWR080" H 1500 2000 50  0001 C CNN
 F 1 "GND" H 1550 2050 50  0000 C CNN
 F 2 "" H 1500 2250 50  0001 C CNN
@@
 $EndBitmap
 $Comp
-L LED:WS2812B D?
+L LED:WS2812B D8
 U 1 1 5CF3B1DC
 P 2550 2500
-F 0 "D?" H 2900 2550 50  0000 L CNN
+F 0 "D8" H 2900 2550 50  0000 L CNN
 F 1 "WS2812B" H 2900 2500 50  0000 L CNN
 F 2 "LED_SMD:LED_WS2812B_PLCC4_5.0x5.0mm_P3.2mm" H 2600 2200 50  0001 L TNN
@@
 $EndComp
 $Comp
-L LED:WS2812B D?
+L LED:WS2812B D9
 U 1 1 5CF3C1DB
 P 3550 2500
-F 0 "D?" H 3900 2550 50  0000 L CNN
+F 0 "D9" H 3900 2550 50  0000 L CNN
 F 1 "WS2812B" H 3900 2500 50  0000 L CNN
 F 2 "LED_SMD:LED_WS2812B_PLCC4_5.0x5.0mm_P3.2mm" H 3600 2200 50  0001 L TNN
@@
 	3850 2500 4250 2500
 $Comp
-L LED:WS2812B D?
+L LED:WS2812B D10
 U 1 1 5CF3CB01
 P 4550 2500
-F 0 "D?" H 4900 2550 50  0000 L CNN
+F 0 "D10" H 4900 2550 50  0000 L CNN
 F 1 "WS2812B" H 4900 2500 50  0000 L CNN
 F 2 "LED_SMD:LED_WS2812B_PLCC4_5.0x5.0mm_P3.2mm" H 4600 2200 50  0001 L TNN
@@
 Wire Wire Line
 	2400 1900 2550 1900
+NoConn ~ 4850 2500
 $EndSCHEMATC

Commit message: update DRC ok,
Parts:
- D10, D8, D9: footprint LED_SMD:LED_WS2812B_PLCC4_5.0x5.0mm_P3.2mm -> footprint-lib:LED_WS2812B_5050_white
Changed lines of the file:
@@
 F 0 "D8" H 2900 2550 50  0000 L CNN
 F 1 "WS2812B" H 2900 2500 50  0000 L CNN
-F 2 "LED_SMD:LED_WS2812B_PLCC4_5.0x5.0mm_P3.2mm" H 2600 2200 50  0001 L TNN
+F 2 "footprint-lib:LED_WS2812B_5050_white" H 2600 2200 50  0001 L TNN
 F 3 "https://cdn-shop.adafruit.com/datasheets/WS2812B.pdf" H 2650 2125 50  0001 L TNN
 	1    2550 2500
@@
 F 0 "D9" H 3900 2550 50  0000 L CNN
 F 1 "WS2812B" H 3900 2500 50  0000 L CNN
-F 2 "LED_SMD:LED_WS2812B_PLCC4_5.0x5.0mm_P3.2mm" H 3600 2200 50  0001 L TNN
+F 2 "footprint-lib:LED_WS2812B_5050_white" H 3600 2200 50  0001 L TNN
 F 3 "https://cdn-shop.adafruit.com/datasheets/WS2812B.pdf" H 3650 2125 50  0001 L TNN
 	1    3550 2500
@@
 F 0 "D10" H 4900 2550 50  0000 L CNN
 F 1 "WS2812B" H 4900 2500 50  0000 L CNN
-F 2 "LED_SMD:LED_WS2812B_PLCC4_5.0x5.0mm_P3.2mm" H 4600 2200 50  0001 L TNN
+F 2 "footprint-lib:LED_WS2812B_5050_white" H 4600 2200 50  0001 L TNN
 F 3 "https://cdn-shop.adafruit.com/datasheets/WS2812B.pdf" H 4650 2125 50  0001 L TNN
 	1    4550 2500
