File: hardware/esp12-lora-remote-station.kicad_pcb (KiCad board)
At the start: 2 copper layers, 95 x 95 mm, 104 parts, among them J1 LM75_HEADER, J10 ROT_ENC_HEADER, J11 I2C_HEADER,2.54, J12 5V_header, J13 5V_header, J2 I2C_HEADER,2.54, J3 P0_HEADER, J4 P1_HEADER, J5 I2C_HEADER,2.54, J6 I2C_HEADER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

Commit message: update manual rout,
Parts:
- turned R24 to 270 degrees
Routing:
- net /esp12_core/usb_to_uart/D_N: track 0.00 -> 29.9 mm, vias 0 -> 2
- net /esp12_core/usb_to_uart/D_P: track 0.00 -> 29.7 mm, vias 0 -> 2
- net Net-(JP7-Pad2): track 17.5 -> 39.0 mm, vias 2 -> 3
- net +5V: track 195.1 -> 215.3 mm, vias 4 -> 7
- net Net-(R20-Pad2): track 19.8 -> 24.9 mm
- net /esp12_core/GPIO13: track 45.3 -> 40.5 mm, vias 0 -> 2
- net +3V3: track 435.7 -> 440.3 mm, vias 4 -> 5
- net /SDA: track 270.0 -> 273.9 mm
- net GND: track 610.4 -> 614.1 mm
- net /esp12_core/nRST: track 106.8 -> 104.2 mm, vias 2 -> 4
- net /esp12_core/GPIO2: track 74.6 -> 77.0 mm, vias 2 -> 4
- net /SCL: track 278.4 -> 275.9 mm, vias 3 -> 5
- net /user_button/B: track 67.5 -> 69.7 mm
- net /esp12_core/GPIO0: track 103.8 -> 101.7 mm, vias 2 -> 4
- net /esp12_core/RXD0: track 75.4 -> 77.4 mm
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Other:
- net class 500mA: clearance 0.4 -> 0.2; trace_width 0.25 -> 0.4
- net class 800mA: clearance 0.4 -> 0.2; trace_width 0.25 -> 0.4

Commit message: update manual rout,
Routing:
- net +3V3: track 440.3 -> 432.4 mm, vias 5 -> 7
- net /SDA: track 273.9 -> 269.2 mm, vias 6 -> 7
Changed lines of the file:
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@@
     (thickness 1.6)
     (drawings 8)
-    (tracks 1107)
+    (tracks 1106)
     (zones 0)
     (modules 104)
@@
   (segment (start 54.642 118.023) (end 54.642 120.317) (width 0.25) (layer F.Cu) (net 3))
   (segment (start 54.642 120.317) (end 54.75 120.425) (width 0.25) (layer F.Cu) (net 3))
-  (segment (start 138.8881 110.4827) (end 144.0274 105.3434) (width 0.25) (layer F.Cu) (net 3))
-  (segment (start 144.0274 105.3434) (end 144.0274 104.6423) (width 0.25) (layer F.Cu) (net 3))
-  (segment (start 144.0274 104.6423) (end 137.3629 97.9778) (width 0.25) (layer F.Cu) (net 3))
-  (segment (start 137.3629 97.9778) (end 133.1472 97.9778) (width 0.25) (layer F.Cu) (net 3))
-  (segment (start 133.1472 97.9778) (end 132.125 99) (width 0.25) (layer F.Cu) (net 3))
-  (segment (start 134 107.875) (end 136.6077 110.4827) (width 0.25) (layer F.Cu) (net 3))
-  (segment (start 136.6077 110.4827) (end 138.8881 110.4827) (width 0.25) (layer F.Cu) (net 3))
-  (segment (start 141 113) (end 140.5313 113) (width 0.25) (layer F.Cu) (net 3))
-  (segment (start 140.5313 113) (end 138.8881 111.3568) (width 0.25) (layer F.Cu) (net 3))
-  (segment (start 138.8881 111.3568) (end 138.8881 110.4827) (width 0.25) (layer F.Cu) (net 3))
   (segment (start 132 107.75) (end 133.875 107.75) (width 0.25) (layer F.Cu) (net 3))
   (segment (start 133.875 107.75) (end 134 107.875) (width 0.25) (layer F.Cu) (net 3))
@@
   (segment (start 117.4792 52.6792) (end 104.8379 52.6792) (width 0.25) (layer F.Cu) (net 3))
   (segment (start 135.1769 52.6792) (end 131.9208 52.6792) (width 0.25) (layer F.Cu) (net 3))
+  (via (at 132.125 99) (size 0.8) (drill 0.4) (layers F.Cu B.Cu) (net 3))
+  (segment (start 134 107.875) (end 133.999986 107.875) (width 0.25) (layer F.Cu) (net 3))
+  (via (at 133.999986 107.875) (size 0.8) (drill 0.4) (layers F.Cu B.Cu) (net 3))
+  (segment (start 130.475 107.875) (end 133.999986 107.875) (width 0.25) (layer B.Cu) (net 3))
+  (segment (start 129.4 106.8) (end 130.475 107.875) (width 0.25) (layer B.Cu) (net 3))
+  (segment (start 132.125 99) (end 129.4 101.725) (width 0.25) (layer B.Cu) (net 3))
+  (segment (start 129.4 101.725) (end 129.4 106.8) (width 0.25) (layer B.Cu) (net 3))
+  (segment (start 141 113) (end 136.2 113) (width 0.25) (layer F.Cu) (net 3))
+  (segment (start 134 110.8) (end 134 107.875) (width 0.25) (layer F.Cu) (net 3))
+  (segment (start 136.2 113) (end 134 110.8) (width 0.25) (layer F.Cu) (net 3))
   (segment (start 117.06 129) (end 117.06 128.3747) (width 0.25) (layer F.Cu) (net 4))
   (segment (start 117.06 128.3747) (end 116.9771 128.3747) (width 0.25) (layer F.Cu) (net 4))
@@
   (segment (start 57.125 101) (end 56.66 100.535) (width 0.25) (layer F.Cu) (net 39))
   (segment (start 56.66 100.535) (end 54.115 100.535) (width 0.25) (layer F.Cu) (net 39))
-  (segment (start 139 105) (end 139 103.8247) (width 0.25) (layer F.Cu) (net 39))
-  (segment (start 134.55 103.95) (end 135.6098 103.95) (width 0.25) (layer F.Cu) (net 39))
-  (segment (start 135.6098 103.95) (end 138.2952 101.2646) (width 0.25) (layer F.Cu) (net 39))
-  (segment (start 138.2952 101.2646) (end 139.4674 101.2646) (width 0.25) (layer F.Cu) (net 39))
-  (segment (start 139.4674 101.2646) (end 140.1753 101.9725) (width 0.25) (layer F.Cu) (net 39))
-  (segment (start 140.1753 101.9725) (end 140.1753 103.0168) (width 0.25) (layer F.Cu) (net 39))
-  (segment (start 140.1753 103.0168) (end 139.3674 103.8247) (width 0.25) (layer F.Cu) (net 39))
-  (segment (start 139.3674 103.8247) (end 139 103.8247) (width 0.25) (layer F.Cu) (net 39))
   (segment (start 139 105) (end 143.0621 105) (width 0.25) (layer F.Cu) (net 39))
-  (segment (start 131.81 68) (end 143.0621 79.2521) (width 0.25) (layer B.Cu) (net 39))
-  (segment (start 143.0621 79.2521) (end 143.0621 105) (width 0.25) (layer B.Cu) (net 39))
   (segment (start 74 87) (end 85.959 87) (width 0.25) (layer F.Cu) (net 39))
   (segment (start 100.2354 64.96) (end 100.1753 64.9) (width 0.25) (layer F.Cu) (net 39))
@@
   (segment (start 69.125 86.2014) (end 69.125 86) (width 0.25) (layer F.Cu) (net 39))
   (segment (start 54.115 100.535) (end 55.2903 100.535) (width 0.25) (layer B.Cu) (net 39))
-  (segment (start 139 105) (end 137.8247 105) (width 0.25) (layer F.Cu) (net 39))
-  (segment (start 137.8247 105) (end 136.6997 106.125) (width 0.25) (layer F.Cu) (net 39))
-  (segment (start 136.6997 106.125) (end 134 106.125) (width 0.25) (layer F.Cu) (net 39))
   (segment (start 59.01 122.2997) (end 58.3747 122.2997) (width 0.25) (layer F.Cu) (net 39))
   (segment (start 58.3747 122.2997) (end 56.5 120.425) (width 0.25) (layer F.Cu) (net 39))
@@
   (segment (start 98.6 64.9) (end 100.1753 64.9) (width 0.25) (layer F.Cu) (net 39))
   (segment (start 106 72) (end 104.8247 72) (width 0.25) (layer F.Cu) (net 39))
-  (segment (start 141 133.08) (end 141 131.9047) (width 0.25) (layer B.Cu) (net 39))
-  (segment (start 141 131.9047) (end 140.6327 131.9047) (width 0.25) (layer B.Cu) (net 39))
-  (segment (start 140.6327 131.9047) (end 139 130.272) (width 0.25) (layer B.Cu) (net 39))
-  (segment (start 139 130.272) (end 139 105) (width 0.25) (layer B.Cu) (net 39))
   (segment (start 59.01 123.175) (end 59.01 122.2997) (width 0.25) (layer F.Cu) (net 39))
   (segment (start 108.2247 54.09) (end 107.1147 55.2) (width 0.25) (layer F.Cu) (net 39))
@@
   (segment (start 109.4 54.09) (end 111.6 56.29) (width 0.25) (layer B.Cu) (net 39))
   (segment (start 111.6 56.29) (end 111.6 70.2) (width 0.25) (layer B.Cu) (net 39))
+  (segment (start 131.81 68) (end 131.81 90.21) (width 0.25) (layer B.Cu) (net 39))
+  (segment (start 143.0621 101.4621) (end 143.0621 104.434315) (width 0.25) (layer B.Cu) (net 39))
+  (segment (start 143.0621 104.434315) (end 143.0621 105) (width 0.25) (layer B.Cu) (net 39))
+  (segment (start 131.81 90.21) (end 143.0621 101.4621) (width 0.25) (layer B.Cu) (net 39))
+  (segment (start 139 105) (end 137.526996 105) (width 0.25) (layer F.Cu) (net 39))
+  (segment (start 137.526996 105) (end 136.401996 106.125) (width 0.25) (layer F.Cu) (net 39))
+  (segment (start 136.401996 106.125) (end 134.575 106.125) (width 0.25) (layer F.Cu) (net 39))
+  (segment (start 134.575 106.125) (end 134 106.125) (width 0.25) (layer F.Cu) (net 39))
+  (via (at 136.2 102.4) (size 0.8) (drill 0.4) (layers F.Cu B.Cu) (net 39))
+  (segment (start 136.2 102.575) (end 136.2 102.4) (width 0.25) (layer F.Cu) (net 39))
+  (segment (start 134.55 103.95) (end 134.825 103.95) (width 0.25) (layer F.Cu) (net 39))
+  (segment (start 134.825 103.95) (end 136.2 102.575) (width 0.25) (layer F.Cu) (net 39))
+  (segment (start 138.8 105) (end 139 105) (width 0.25) (layer B.Cu) (net 39))
+  (segment (start 136.2 102.4) (end 138.8 105) (width 0.25) (layer B.Cu) (net 39))
+  (segment (start 139 131.08) (end 141 133.08) (width 0.25) (layer B.Cu) (net 39))
+  (segment (start 139 105) (end 139 131.08) (width 0.25) (layer B.Cu) (net 39))
   (segment (start 54.115 103.075) (end 54.115 104.2503) (width 0.25) (layer B.Cu) (net 40))
   (segment (start 54.115 104.2503) (end 53.0079 105.3574) (width 0.25) (layer B.Cu) (net 40))
@@
   (segment (start 106 68.2847) (end 105.56 68.2847) (width 0.25) (layer F.Cu) (net 40))
   (segment (start 105.56 68.2847) (end 100.1753 62.9) (width 0.25) (layer F.Cu) (net 40))
-  (segment (start 139 102.46) (end 139 103.6353) (width 0.25) (layer B.Cu) (net 40))
-  (segment (start 141 130.54) (end 141 129.3647) (width 0.25) (layer B.Cu) (net 40))
-  (segment (start 141 129.3647) (end 140.192 129.3647) (width 0.25) (layer B.Cu) (net 40))
-  (segment (start 140.192 129.3647) (end 139.8246 128.9973) (width 0.25) (layer B.Cu) (net 40))
-  (segment (start 139.8246 128.9973) (end 139.8246 116.8633) (width 0.25) (layer B.Cu) (net 40))
-  (segment (start 139.8246 116.8633) (end 140.1753 116.5126) (width 0.25) (layer B.Cu) (net 40))
-  (segment (start 140.1753 116.5126) (end 140.1753 104.0025) (width 0.25) (layer B.Cu) (net 40))
-  (segment (start 140.1753 104.0025) (end 139.8081 103.6353) (width 0.25) (layer B.Cu) (net 40))
-  (segment (start 139.8081 103.6353) (end 139 103.6353) (width 0.25) (layer B.Cu) (net 40))
   (segment (start 108.2247 56.63) (end 107.5947 56) (width 0.25) (layer F.Cu) (net 40))
   (segment (start 107.5947 56) (end 106.25 56) (width 0.25) (layer F.Cu) (net 40))
@@
   (segment (start 102.6091 61.1909) (end 103.1909 61.1909) (width 0.25) (layer F.Cu) (net 40))
   (segment (start 103.1909 61.1909) (end 106 64) (width 0.25) (layer F.Cu) (net 40))
+  (segment (start 139.45001 128.99001) (end 141 130.54) (width 0.25) (layer B.Cu) (net 40))
+  (segment (start 139.45001 106.175001) (end 139.45001 128.99001) (width 0.25) (layer B.Cu) (net 40))
+  (segment (start 140.110001 106.175001) (end 139.45001 106.175001) (width 0.25) (layer B.Cu) (net 40))
+  (segment (start 139 102.46) (end 139.4 102.86) (width 0.25) (layer B.Cu) (net 40))
+  (segment (start 140.175001 103.889999) (end 140.175001 106.110001) (width 0.25) (layer B.Cu) (net 40))
+  (segment (start 139.4 103.824999) (end 140.110001 103.824999) (width 0.25) (layer B.Cu) (net 40))
+  (segment (start 139.4 102.86) (end 139.4 103.824999) (width 0.25) (layer B.Cu) (net 40))
+  (segment (start 140.110001 103.824999) (end 140.175001 103.889999) (width 0.25) (layer B.Cu) (net 40))
+  (segment (start 140.175001 106.110001) (end 140.110001 106.175001) (width 0.25) (layer B.Cu) (net 40))
   (segment (start 106.25 56.8) (end 107.0253 56.8) (width 0.25) (layer F.Cu) (net 41))
   (segment (start 109.4 59.17) (end 108.2247 59.17) (width 0.25) (layer F.Cu) (net 41))

Commit message: update DRC ok,
Parts:
- moved J3 4.89 mm to (54.4, 137.4)
- moved C10 3.10 mm to (101.0, 128.2)
- moved C9 3.10 mm to (99.0, 128.2)
- turned Q1 to 90 degrees
Routing:
- net /esp12_core/usb_to_uart/DTR: track 33.8 -> 25.3 mm, vias 0 -> 2
- net Net-(Q1-Pad1): track 8.79 -> 3.22 mm
- net /digital_input/PO2: track 4.38 -> 9.41 mm
- net /digital_input/PO3: track 3.70 -> 8.62 mm
- net /digital_input/PO6: track 9.93 -> 14.7 mm
- net /digital_input/PO4: track 4.72 -> 9.21 mm
- net /esp12_core/usb_to_uart/D_N: track 29.9 -> 25.4 mm
- net /digital_input/PO1: track 5.86 -> 10.2 mm
- net GND: track 614.1 -> 617.9 mm
- net /digital_input/PO5: track 6.25 -> 9.99 mm
- net /digital_input/PO0: track 7.79 -> 11.0 mm
- net Net-(D10-Pad4): track 19.3 -> 16.8 mm
- net /esp12_core/nRST: track 104.2 -> 106.2 mm
- net /digital_input/PO7: track 11.5 -> 13.6 mm
- net /esp12_core/usb_to_uart/D_P: track 29.7 -> 28.1 mm
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
Commit message: update DRC ok,
Routing:
- net /SCL: track 276.1 -> 284.7 mm
- net /esp12_core/INT: track 4.82 -> 4.13 mm

Commit message: update DRC ok,
Parts:
- D10, D8, D9: footprint LED_SMD:LED_WS2812B_PLCC4_5.0x5.0mm_P3.2mm -> footprint-lib:LED_WS2812B_5050_white

Commit message: update copper pour,
Routing:
- net GND: vias 2 -> 14
- net (no net): vias 0 -> 1
- added copper zone on B.Cu, net GND
- added copper zone on F.Cu, net GND
Changed lines of the file:
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@@
     (thickness 1.6)
     (drawings 8)
-    (tracks 1090)
+    (tracks 1103)
     (zones 0)
     (modules 104)
@@
     (add_net /digital_input/PO6)
     (add_net /digital_input/PO7)
-    (add_net /esp12_core/ADC)
     (add_net /esp12_core/EN)
     (add_net /esp12_core/GPIO0)
@@
     (add_net /esp12_core/INT)
     (add_net /esp12_core/RXD0)
-    (add_net /esp12_core/SPI_CLK)
-    (add_net /esp12_core/SPI_INT)
-    (add_net /esp12_core/SPI_MISO)
-    (add_net /esp12_core/SPI_MOSI)
     (add_net /esp12_core/TXD0)
     (add_net /esp12_core/nRST)
-    (add_net /esp12_core/usb_to_uart/ACTIVE)
-    (add_net /esp12_core/usb_to_uart/CTS)
-    (add_net /esp12_core/usb_to_uart/DCD)
-    (add_net /esp12_core/usb_to_uart/DSR)
     (add_net /esp12_core/usb_to_uart/DTR)
     (add_net /esp12_core/usb_to_uart/D_N)
     (add_net /esp12_core/usb_to_uart/D_P)
-    (add_net /esp12_core/usb_to_uart/OTG_ID)
-    (add_net /esp12_core/usb_to_uart/RI)
     (add_net /esp12_core/usb_to_uart/RTS)
     (add_net /user_button/A)
@@
     (add_net "Net-(C1-Pad1)")
     (add_net "Net-(D1-Pad2)")
-    (add_net "Net-(D10-Pad2)")
     (add_net "Net-(D10-Pad4)")
     (add_net "Net-(D2-Pad2)")
@@
     (add_net "Net-(R32-Pad1)")
     (add_net "Net-(R33-Pad1)")
-    (add_net "Net-(RN1-Pad4)")
-    (add_net "Net-(RN1-Pad5)")
-    (add_net "Net-(U2-Pad3)")
-    (add_net "Net-(U2-Pad4)")
-    (add_net "Net-(U7-Pad10)")
-    (add_net "Net-(U7-Pad12)")
-    (add_net "Net-(U7-Pad13)")
-    (add_net "Net-(U7-Pad14)")
-    (add_net "Net-(U7-Pad15)")
-    (add_net "Net-(U7-Pad16)")
-    (add_net "Net-(U7-Pad17)")
-    (add_net "Net-(U7-Pad18)")
-    (add_net "Net-(U7-Pad19)")
-    (add_net "Net-(U7-Pad20)")
-    (add_net "Net-(U7-Pad21)")
-    (add_net "Net-(U7-Pad22)")
-    (add_net "Net-(U7-Pad9)")
   )
   (net_class 500mA ""
@@
   (gr_line (start 145 140) (end 145 55) (layer Edge.Cuts) (width 0.05))
   (gr_line (start 50 55) (end 50 140) (layer Edge.Cuts) (width 0.05))
+  (via (at 69.8 116) (size 0.8) (drill 0.4) (layers F.Cu B.Cu) (net 1))
+  (via (at 66.2 116.2) (size 0.8) (drill 0.4) (layers F.Cu B.Cu) (net 1))
+  (via (at 64.4 115.4) (size 0.8) (drill 0.4) (layers F.Cu B.Cu) (net 0))
   (segment (start 140.9998 120.7877) (end 141 120.788) (width 0.25) (layer F.Cu) (net 1))
   (segment (start 141 120.788) (end 139.762 122.025) (width 0.25) (layer F.Cu) (net 1))
@@
   (segment (start 129.8 105) (end 131.6325 105) (width 0.25) (layer F.Cu) (net 1))
   (segment (start 129.718 105.082) (end 129.8 105) (width 0.25) (layer F.Cu) (net 1))
+  (via (at 115 60) (size 0.8) (drill 0.4) (layers F.Cu B.Cu) (net 1))
+  (via (at 70 80) (size 0.8) (drill 0.4) (layers F.Cu B.Cu) (net 1))
+  (via (at 105 132) (size 0.8) (drill 0.4) (layers F.Cu B.Cu) (net 1))
+  (via (at 68 134) (size 0.8) (drill 0.4) (layers F.Cu B.Cu) (net 1))
+  (via (at 66 135) (size 0.8) (drill 0.4) (layers F.Cu B.Cu) (net 1))
+  (via (at 63 135) (size 0.8) (drill 0.4) (layers F.Cu B.Cu) (net 1))
+  (via (at 61 135) (size 0.8) (drill 0.4) (layers F.Cu B.Cu) (net 1))
+  (via (at 58 135) (size 0.8) (drill 0.4) (layers F.Cu B.Cu) (net 1))
+  (via (at 65.6 121) (size 0.8) (drill 0.4) (layers F.Cu B.Cu) (net 1))
+  (via (at 132.2 55) (size 0.8) (drill 0.4) (layers F.Cu B.Cu) (net 1))
   (segment (start 64.2625 87) (end 67 87) (width 0.25) (layer F.Cu) (net 2))
   (segment (start 64.2625 87) (end 64.2625 87.06) (width 0.25) (layer F.Cu) (net 2))
@@
   (via (at 105 61.8) (size 0.8) (layers F.Cu B.Cu) (net 73))
   (via (at 104.774 120.347) (size 0.8) (layers F.Cu B.Cu) (net 73))
+  (zone (net 1) (net_name GND) (layer F.Cu) (hatch edge 0.508)
+    (connect_pads (clearance 0.508))
+    (min_thickness 0.254)
+    (fill yes (arc_segments 32) (thermal_gap 0.508) (thermal_bridge_width 0.508))
+    (polygon
+      (pts
+        (xy 45 45) (xy 45 150) (xy 150 150) (xy 150 45)
+      )
+    )
+  )
+  (zone (net 1) (net_name GND) (layer B.Cu) (hatch edge 0.508)
+    (connect_pads (clearance 0.508))
+    (min_thickness 0.254)
+    (fill yes (arc_segments 32) (thermal_gap 0.508) (thermal_bridge_width 0.508))
+    (polygon
+      (pts
+        (xy 45 45) (xy 45 150) (xy 150 150) (xy 150 45)
+      )
+    )
+  )
 )
