File: hardware/esp12-lora-remote-station.kicad_pcb (KiCad board)
At the start: 2 copper layers, 95 x 95 mm, 104 parts, among them J1 LM75_HEADER, J10 ROT_ENC_HEADER, J11 I2C_HEADER,2.54, J12 5V_header, J13 5V_header, J2 I2C_HEADER,2.54, J3 P0_HEADER, J4 P1_HEADER, J5 I2C_HEADER,2.54, J6 I2C_HEADER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

Commit message: send to fab,
Parts:
- turned R22 to 270 degrees
- turned R23 to 270 degrees
Routing:
- net /esp12_core/GPIO2: track 77.0 -> 74.2 mm
- net /esp12_core/GPIO15: track 48.8 -> 46.1 mm
- net Net-(R23-Pad2): track 6.66 -> 6.04 mm
- net GND: vias 14 -> 16
Changed lines of the file:
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@@
     (thickness 1.6)
     (drawings 8)
-    (tracks 1103)
+    (tracks 1102)
     (zones 0)
     (modules 104)
@@
       (outputformat 1)
       (mirror false)
-      (drillshape 1)
+      (drillshape 0)
       (scaleselection 1)
-      (outputdirectory ""))
+      (outputdirectory "esp8266_remote_monitor/"))
   )
   (net 0 "")
@@
     (tags "SPST button tactile switch")
     (attr smd)
-    (fp_text reference SW5 (at 0 -2.6 90) (layer F.SilkS)
+    (fp_text reference SW5 (at 0 3.2 90) (layer F.SilkS)
       (effects (font (size 1 1) (thickness 0.15)))
     )
@@
     (tags "resistor handsolder")
     (attr smd)
-    (fp_text reference R24 (at 0 -1.43 90) (layer F.SilkS)
+    (fp_text reference R24 (at 3.325 0 90) (layer F.SilkS)
       (effects (font (size 1 1) (thickness 0.15)))
     )
@@
   )
   (module Resistor_SMD:R_0603_1608Metric_Pad1.05x0.95mm_HandSolder (layer F.Cu)
-    (at 82 100.875 90)
+    (at 82 100.875 270)
     (descr "Resistor SMD 0603 (1608 Metric), square (rectangular) end terminal, IPC_7351 nominal with elongated pad for handsoldering. (Body size source: http://www.tortai-tech.com/upload/download/2011102023233369053.pdf), generated with kicad-footprint-generator")
     (tags "resistor handsolder")
@@
     (fp_line (start -0.8 -0.4) (end 0.8 -0.4) (layer F.Fab) (width 0.1))
     (fp_line (start -0.8 0.4) (end -0.8 -0.4) (layer F.Fab) (width 0.1))
-    (pad 2 smd roundrect (at 0.875 0 90) (size 1.05 0.95) (layers F.Cu F.Paste F.Mask) (roundrect_rratio 0.25)
+    (pad 2 smd roundrect (at 0.875 0 270) (size 1.05 0.95) (layers F.Cu F.Paste F.Mask) (roundrect_rratio 0.25)
       (net 62 "Net-(R23-Pad2)"))
-    (pad 1 smd roundrect (at -0.875 0 90) (size 1.05 0.95) (layers F.Cu F.Paste F.Mask) (roundrect_rratio 0.25)
+    (pad 1 smd roundrect (at -0.875 0 270) (size 1.05 0.95) (layers F.Cu F.Paste F.Mask) (roundrect_rratio 0.25)
       (net 63 /esp12_core/GPIO15))
     (model ${KISYS3DMOD}/Resistor_SMD.3dshapes/R_0603_1608Metric.wrl
@@
   )
   (module Resistor_SMD:R_0603_1608Metric_Pad1.05x0.95mm_HandSolder (layer F.Cu)
-    (at 74 101 90)
+    (at 74 101 270)
     (descr "Resistor SMD 0603 (1608 Metric), square (rectangular) end terminal, IPC_7351 nominal with elongated pad for handsoldering. (Body size source: http://www.tortai-tech.com/upload/download/2011102023233369053.pdf), generated with kicad-footprint-generator")
     (tags "resistor handsolder")
@@
     (fp_line (start -0.8 -0.4) (end 0.8 -0.4) (layer F.Fab) (width 0.1))
     (fp_line (start -0.8 0.4) (end -0.8 -0.4) (layer F.Fab) (width 0.1))
-    (pad 2 smd roundrect (at 0.875 0 90) (size 1.05 0.95) (layers F.Cu F.Paste F.Mask) (roundrect_rratio 0.25)
+    (pad 2 smd roundrect (at 0.875 0 270) (size 1.05 0.95) (layers F.Cu F.Paste F.Mask) (roundrect_rratio 0.25)
       (net 61 "Net-(R22-Pad2)"))
-    (pad 1 smd roundrect (at -0.875 0 90) (size 1.05 0.95) (layers F.Cu F.Paste F.Mask) (roundrect_rratio 0.25)
+    (pad 1 smd roundrect (at -0.875 0 270) (size 1.05 0.95) (layers F.Cu F.Paste F.Mask) (roundrect_rratio 0.25)
       (net 55 /esp12_core/GPIO2))
     (model ${KISYS3DMOD}/Resistor_SMD.3dshapes/R_0603_1608Metric.wrl
@@
   (via (at 65.6 121) (size 0.8) (drill 0.4) (layers F.Cu B.Cu) (net 1))
   (via (at 132.2 55) (size 0.8) (drill 0.4) (layers F.Cu B.Cu) (net 1))
+  (via (at 78.6 88.4) (size 0.8) (drill 0.4) (layers F.Cu B.Cu) (net 1))
+  (via (at 87.6 88.6) (size 0.8) (drill 0.4) (layers F.Cu B.Cu) (net 1))
   (segment (start 64.2625 87) (end 67 87) (width 0.25) (layer F.Cu) (net 2))
   (segment (start 64.2625 87) (end 64.2625 87.06) (width 0.25) (layer F.Cu) (net 2))
@@
   (segment (start 97.85 68.9) (end 96.2 70.55) (width 0.25) (layer F.Cu) (net 55))
   (segment (start 96.2 70.55) (end 96.2 71.6) (width 0.25) (layer F.Cu) (net 55))
-  (segment (start 76.5543 96.9248) (end 75.8685 96.9248) (width 0.25) (layer F.Cu) (net 55))
-  (segment (start 75.8685 96.9248) (end 73.1575 99.6358) (width 0.25) (layer F.Cu) (net 55))
-  (segment (start 73.1575 99.6358) (end 73.1575 101.032) (width 0.25) (layer F.Cu) (net 55))
-  (segment (start 73.1575 101.032) (end 74 101.875) (width 0.25) (layer F.Cu) (net 55))
   (via (at 77 69.875) (size 0.8) (layers F.Cu B.Cu) (net 55))
   (via (at 80 64) (size 0.8) (layers F.Cu B.Cu) (net 55))
   (via (at 96.2 71.6) (size 0.8) (layers F.Cu B.Cu) (net 55))
   (via (at 76.5543 96.9248) (size 0.8) (layers F.Cu B.Cu) (net 55))
+  (segment (start 74 99.4791) (end 76.5543 96.9248) (width 0.25) (layer F.Cu) (net 55))
+  (segment (start 74 100.125) (end 74 99.4791) (width 0.25) (layer F.Cu) (net 55))
   (segment (start 77.1731 65.1209) (end 78.4 66.3478) (width 0.25) (layer B.Cu) (net 56))
   (segment (start 78.4 66.3478) (end 78.4 73.6481) (width 0.25) (layer B.Cu) (net 56))
@@
   (via (at 111.8 78.8) (size 0.8) (layers F.Cu B.Cu) (net 60))
   (via (at 108.471 91.4215) (size 0.8) (layers F.Cu B.Cu) (net 60))
-  (segment (start 78 104.9) (end 78 103.825) (width 0.25) (layer F.Cu) (net 61))
-  (segment (start 78 103.825) (end 77.6997 103.825) (width 0.25) (layer F.Cu) (net 61))
-  (segment (start 77.6997 103.825) (end 74 100.125) (width 0.25) (layer F.Cu) (net 61))
-  (segment (start 86 104.9) (end 86 103.825) (width 0.25) (layer F.Cu) (net 62))
-  (segment (start 86 103.825) (end 85.8247 103.825) (width 0.25) (layer F.Cu) (net 62))
-  (segment (start 85.8247 103.825) (end 82 100) (width 0.25) (layer F.Cu) (net 62))
-  (segment (start 82 101.75) (end 81.1799 100.93) (width 0.25) (layer F.Cu) (net 63))
-  (segment (start 81.1799 100.93) (end 81.1799 99.4556) (width 0.25) (layer F.Cu) (net 63))
-  (segment (start 81.1799 99.4556) (end 82.4262 98.2093) (width 0.25) (layer F.Cu) (net 63))
-  (segment (start 82.4262 98.2093) (end 89.9177 98.2093) (width 0.25) (layer F.Cu) (net 63))
+  (segment (start 74 101.875) (end 74 104.8) (width 0.25) (layer F.Cu) (net 61))
+  (segment (start 74.1 104.9) (end 78 104.9) (width 0.25) (layer F.Cu) (net 61))
+  (segment (start 74 104.8) (end 74.1 104.9) (width 0.25) (layer F.Cu) (net 61))
+  (segment (start 82 101.75) (end 82 103) (width 0.25) (layer F.Cu) (net 62))
+  (segment (start 83.9 104.9) (end 86 104.9) (width 0.25) (layer F.Cu) (net 62))
+  (segment (start 82 103) (end 83.9 104.9) (width 0.25) (layer F.Cu) (net 62))
   (segment (start 89.9177 98.2093) (end 90.252 97.875) (width 0.25) (layer F.Cu) (net 63))
   (segment (start 90.252 97.875) (end 91.748 97.875) (width 0.25) (layer F.Cu) (net 63))
@@
   (via (at 101 75.2) (size 0.8) (layers F.Cu B.Cu) (net 63))
   (via (at 95.4799 98.2093) (size 0.8) (layers F.Cu B.Cu) (net 63))
+  (segment (start 82 99) (end 82.7907 98.2093) (width 0.25) (layer F.Cu) (net 63))
+  (segment (start 82 100) (end 82 99) (width 0.25) (layer F.Cu) (net 63))
+  (segment (start 82.7907 98.2093) (end 89.9177 98.2093) (width 0.25) (layer F.Cu) (net 63))
   (segment (start 94 104.9) (end 94 103.9) (width 0.25) (layer F.Cu) (net 64))
   (segment (start 94 103.9) (end 91.85 101.75) (width 0.25) (layer F.Cu) (net 64))
