File: hardware/esp12_core.sch (KiCad schematic (older format))
At the start: 16 parts

Commit message: after DRC,
Parts:
- gave numbers to parts that had none: 16
Connections:
- no-connect marks 2 -> 7

Commit message: after routing,
Parts:
- removed C7: CP10uf,16V, Capacitor_SMD:CP_Elec_4x5.3, symbol taobao-cp:CP10uf,16V
- removed C8: C106,0603, Capacitor_SMD:C_0603_1608Metric_Pad1.05x0.95mm_HandSolder, symbol taobao-c:C106,0603
- removed U5: AMS1117-3.3, footprint-lib:AMS1117_SOT-223, symbol taobao-components:AMS1117-3.3
- J5: footprint Connector_PinHeader_2.54mm:PinHeader_1x02_P2.54mm_Vertical -> footprint-lib:I2C_DEBUG,2.54
- U4: footprint footprint-lib:ESP-12 -> footprint-lib:ESP-12E
Changed lines of the file:
@@
 F 0 "U4" H 3600 6500 50  0000 C CNN
 F 1 "ESP12" H 3600 6400 50  0000 C CNN
-F 2 "footprint-lib:ESP-12" H 3650 4500 50  0001 C CNN
+F 2 "footprint-lib:ESP-12E" H 3650 4500 50  0001 C CNN
 F 3 "" H 3650 4500 50  0001 C CNN
 	1    3600 5200
@@
 Wire Wire Line
 	3600 6050 3600 6200
-$Comp
-L taobao-components:AMS1117-3.3 U?
-U 1 1 5CD48784
-P 8150 5500
-AR Path="/5CD03616/5CD48784" Ref="U?"  Part="1"
-AR Path="/5CD03534/5CD48784" Ref="U?"  Part="1"
-AR Path="/5CD47361/5CD48784" Ref="U?"  Part="1"
-AR Path="/5CF23C1A/5CD48784" Ref="U5"  Part="1"
-F 0 "U5" H 8150 5742 50  0000 C CNN
-F 1 "AMS1117-3.3" H 8150 5651 50  0000 C CNN
-F 2 "footprint-lib:AMS1117_SOT-223" H 8150 5700 50  0001 C CNN
-F 3 "" H 8250 5250 50  0001 C CNN
-	1    8150 5500
-	1    0    0    -1
-$EndComp
-$Comp
-L power:+5V #PWR?
-U 1 1 5CD4878A
-P 7500 5300
-AR Path="/5CD03616/5CD4878A" Ref="#PWR?"  Part="1"
-AR Path="/5CD03534/5CD4878A" Ref="#PWR?"  Part="1"
-AR Path="/5CD47361/5CD4878A" Ref="#PWR?"  Part="1"
-AR Path="/5CF23C1A/5CD4878A" Ref="#PWR039"  Part="1"
-F 0 "#PWR039" H 7500 5150 50  0001 C CNN
-F 1 "+5V" H 7550 5500 50  0000 C CNN
-F 2 "" H 7500 5300 50  0001 C CNN
-F 3 "" H 7500 5300 50  0001 C CNN
-	1    7500 5300
-	1    0    0    -1
-$EndComp
-$Comp
-L power:+3V3 #PWR?
-U 1 1 5CD48790
-P 8750 5300
-AR Path="/5CD03616/5CD48790" Ref="#PWR?"  Part="1"
-AR Path="/5CD03534/5CD48790" Ref="#PWR?"  Part="1"
-AR Path="/5CD47361/5CD48790" Ref="#PWR?"  Part="1"
-AR Path="/5CF23C1A/5CD48790" Ref="#PWR040"  Part="1"
-F 0 "#PWR040" H 8750 5150 50  0001 C CNN
-F 1 "+3V3" H 8800 5500 50  0000 C CNN
-F 2 "" H 8750 5300 50  0001 C CNN
-F 3 "" H 8750 5300 50  0001 C CNN
-	1    8750 5300
-	1    0    0    -1
-$EndComp
-$Comp
-L taobao-cp:CP10uf,16V C?
-U 1 1 5CD48796
-P 7500 5700
-AR Path="/5CD03616/5CD48796" Ref="C?"  Part="1"
-AR Path="/5CD03534/5CD48796" Ref="C?"  Part="1"
-AR Path="/5CD47361/5CD48796" Ref="C?"  Part="1"
-AR Path="/5CF23C1A/5CD48796" Ref="C7"  Part="1"
-F 0 "C7" H 7600 5750 50  0000 L CNN
-F 1 "CP10uf,16V" H 7600 5700 50  0000 L CNN
-F 2 "Capacitor_SMD:CP_Elec_4x5.3" H 7500 5700 50  0001 C CNN
-F 3 "~" H 7500 5700 50  0001 C CNN
-	1    7500 5700
-	1    0    0    -1
-$EndComp
-$Comp
-L taobao-c:C106,0603 C?
-U 1 1 5CD4879C
-P 8750 5700
-AR Path="/5CD03616/5CD4879C" Ref="C?"  Part="1"
-AR Path="/5CD03534/5CD4879C" Ref="C?"  Part="1"
-AR Path="/5CD47361/5CD4879C" Ref="C?"  Part="1"
-AR Path="/5CF23C1A/5CD4879C" Ref="C8"  Part="1"
-F 0 "C8" H 8850 5750 50  0000 L CNN
-F 1 "C106,0603" H 8850 5700 50  0000 L CNN
-F 2 "Capacitor_SMD:C_0603_1608Metric_Pad1.05x0.95mm_HandSolder" H 8750 5700 50  0001 C CNN
-F 3 "~" H 8750 5700 50  0001 C CNN
-	1    8750 5700
-	1    0    0    -1
-$EndComp
-Wire Wire Line
-	7500 5300 7500 5500
-Wire Wire Line
-	7850 5500 7500 5500
-Connection ~ 7500 5500
-Wire Wire Line
-	7500 5500 7500 5600
-$Comp
-L power:GND #PWR?
-U 1 1 5CD487A6
-P 7500 6000
-AR Path="/5CD03616/5CD487A6" Ref="#PWR?"  Part="1"
-AR Path="/5CD03534/5CD487A6" Ref="#PWR?"  Part="1"
-AR Path="/5CD47361/5CD487A6" Ref="#PWR?"  Part="1"
-AR Path="/5CF23C1A/5CD487A6" Ref="#PWR042"  Part="1"
-F 0 "#PWR042" H 7500 5750 50  0001 C CNN
-F 1 "GND" H 7550 5800 50  0000 C CNN
-F 2 "" H 7500 6000 50  0001 C CNN
-F 3 "" H 7500 6000 50  0001 C CNN
-	1    7500 6000
-	1    0    0    -1
-$EndComp
-Wire Wire Line
-	7500 5800 7500 6000
-Wire Wire Line
-	8450 5500 8750 5500
-Wire Wire Line
-	8750 5500 8750 5300
-Wire Wire Line
-	8750 5500 8750 5600
-Connection ~ 8750 5500
-$Comp
-L power:GND #PWR?
-U 1 1 5CD487B1
-P 8750 6000
-AR Path="/5CD03616/5CD487B1" Ref="#PWR?"  Part="1"
-AR Path="/5CD03534/5CD487B1" Ref="#PWR?"  Part="1"
-AR Path="/5CD47361/5CD487B1" Ref="#PWR?"  Part="1"
-AR Path="/5CF23C1A/5CD487B1" Ref="#PWR043"  Part="1"
-F 0 "#PWR043" H 8750 5750 50  0001 C CNN
-F 1 "GND" H 8800 5800 50  0000 C CNN
-F 2 "" H 8750 6000 50  0001 C CNN
-F 3 "" H 8750 6000 50  0001 C CNN
-	1    8750 6000
-	1    0    0    -1
-$EndComp
-Wire Wire Line
-	8750 5800 8750 6000
-$Comp
-L power:GND #PWR?
-U 1 1 5CD487B8
-P 8150 5950
-AR Path="/5CD03616/5CD487B8" Ref="#PWR?"  Part="1"
-AR Path="/5CD03534/5CD487B8" Ref="#PWR?"  Part="1"
-AR Path="/5CD47361/5CD487B8" Ref="#PWR?"  Part="1"
-AR Path="/5CF23C1A/5CD487B8" Ref="#PWR041"  Part="1"
-F 0 "#PWR041" H 8150 5700 50  0001 C CNN
-F 1 "GND" H 8200 5750 50  0000 C CNN
-F 2 "" H 8150 5950 50  0001 C CNN
-F 3 "" H 8150 5950 50  0001 C CNN
-	1    8150 5950
-	1    0    0    -1
-$EndComp
-Wire Wire Line
-	8150 5800 8150 5950
 $Bitmap
 Pos -1250 1550
@@
 F 0 "J5" H 1222 1132 50  0000 R CNN
 F 1 "I2C_HEADER,2.54" H 1222 1223 50  0000 R CNN
-F 2 "Connector_PinHeader_2.54mm:PinHeader_1x02_P2.54mm_Vertical" H 1250 800 50  0001 C CNN
+F 2 "footprint-lib:I2C_DEBUG,2.54" H 1250 800 50  0001 C CNN
 F 3 "" H 1250 1150 50  0001 C CNN
 	1    1250 1200

Commit message: update,
Parts:
- added R?: R123,0603, Resistor_SMD:R_0603_1608Metric_Pad1.05x0.95mm_HandSolder, symbol taobao-r:R123,0603
- added TP? (x2): TestPoint, symbol Connector:TestPoint
Connections:
- net GND: now also R?.1
- net GPIO15: now also R?.2
- net RXD0: now also TP?.1
- net TXD0: now also TP?.1
