File: hardware/usb_to_uart.sch (KiCad schematic (older format))
At the start: 11 parts

Commit message: after DRC,
Parts:
- gave numbers to parts that had none: 11
Connections:
- no-connect marks 3 -> 8
Changed lines of the file:
@@
 AR Path="/5CD03534/5CD5414F/5CD5CDC5" Ref="U?"  Part="1"
 AR Path="/5CD47361/5CD5414F/5CD5CDC5" Ref="U?"  Part="1"
-AR Path="/5CF23C1A/5CD5414F/5CD5CDC5" Ref="U?"  Part="1"
-F 0 "U?" H 5050 3050 50  0000 L CNN
+AR Path="/5CF23C1A/5CD5414F/5CD5CDC5" Ref="U7"  Part="1"
+F 0 "U7" H 5050 3050 50  0000 L CNN
 F 1 "CP2102" H 5050 3000 50  0000 L CNN
 F 2 "w_smd_qfn:qfn-28" H 4000 1600 50  0001 C CNN
@@
 AR Path="/5CD03534/5CD5414F/5CD5D577" Ref="#PWR?"  Part="1"
 AR Path="/5CD47361/5CD5414F/5CD5D577" Ref="#PWR?"  Part="1"
-AR Path="/5CF23C1A/5CD5414F/5CD5D577" Ref="#PWR?"  Part="1"
-F 0 "#PWR?" H 3650 1200 50  0001 C CNN
+AR Path="/5CF23C1A/5CD5414F/5CD5D577" Ref="#PWR045"  Part="1"
+F 0 "#PWR045" H 3650 1200 50  0001 C CNN
 F 1 "GND" H 3650 1250 50  0000 C CNN
 F 2 "" H 3650 1450 50  0001 C CNN
@@
 AR Path="/5CD03534/5CD5414F/5CD5DD7B" Ref="R?"  Part="1"
 AR Path="/5CD47361/5CD5414F/5CD5DD7B" Ref="R?"  Part="1"
-AR Path="/5CF23C1A/5CD5414F/5CD5DD7B" Ref="R?"  Part="1"
-F 0 "R?" V 3950 1300 50  0000 C CNN
+AR Path="/5CF23C1A/5CD5414F/5CD5DD7B" Ref="R15"  Part="1"
+F 0 "R15" V 3950 1300 50  0000 C CNN
 F 1 "R471,0603" V 4050 1300 50  0000 C CNN
 F 2 "Resistor_SMD:R_0603_1608Metric_Pad1.05x0.95mm_HandSolder" H 4200 1300 50  0001 C CNN
@@
 AR Path="/5CD03534/5CD5414F/5CD5FC61" Ref="#PWR?"  Part="1"
 AR Path="/5CD47361/5CD5414F/5CD5FC61" Ref="#PWR?"  Part="1"
-AR Path="/5CF23C1A/5CD5414F/5CD5FC61" Ref="#PWR?"  Part="1"
-F 0 "#PWR?" H 1550 3050 50  0001 C CNN
+AR Path="/5CF23C1A/5CD5414F/5CD5FC61" Ref="#PWR049"  Part="1"
+F 0 "#PWR049" H 1550 3050 50  0001 C CNN
 F 1 "+3V3" H 1600 3400 50  0000 C CNN
 F 2 "" H 1550 3200 50  0001 C CNN
@@
 AR Path="/5CD03534/5CD5414F/5CD60483" Ref="C?"  Part="1"
 AR Path="/5CD47361/5CD5414F/5CD60483" Ref="C?"  Part="1"
-AR Path="/5CF23C1A/5CD5414F/5CD60483" Ref="C?"  Part="1"
-F 0 "C?" H 1450 3650 50  0000 R CNN
+AR Path="/5CF23C1A/5CD5414F/5CD60483" Ref="C9"  Part="1"
+F 0 "C9" H 1450 3650 50  0000 R CNN
 F 1 "C106,0603" H 1450 3600 50  0000 R CNN
 F 2 "Capacitor_SMD:C_0603_1608Metric_Pad1.05x0.95mm_HandSolder" H 1550 3600 50  0001 C CNN
@@
 AR Path="/5CD03534/5CD5414F/5CD6081C" Ref="C?"  Part="1"
 AR Path="/5CD47361/5CD5414F/5CD6081C" Ref="C?"  Part="1"
-AR Path="/5CF23C1A/5CD5414F/5CD6081C" Ref="C?"  Part="1"
-F 0 "C?" H 1900 3650 50  0000 L CNN
+AR Path="/5CF23C1A/5CD5414F/5CD6081C" Ref="C10"  Part="1"
+F 0 "C10" H 1900 3650 50  0000 L CNN
 F 1 "C104,0603" H 1900 3600 50  0000 L CNN
 F 2 "Capacitor_SMD:C_0603_1608Metric_Pad1.05x0.95mm_HandSolder" H 1800 3600 50  0001 C CNN
@@
 AR Path="/5CD03534/5CD5414F/5CD6349A" Ref="#PWR?"  Part="1"
 AR Path="/5CD47361/5CD5414F/5CD6349A" Ref="#PWR?"  Part="1"
-AR Path="/5CF23C1A/5CD5414F/5CD6349A" Ref="#PWR?"  Part="1"
-F 0 "#PWR?" H 1700 3750 50  0001 C CNN
+AR Path="/5CF23C1A/5CD5414F/5CD6349A" Ref="#PWR050"  Part="1"
+F 0 "#PWR050" H 1700 3750 50  0001 C CNN
 F 1 "GND" H 1750 3800 50  0000 C CNN
 F 2 "" H 1700 4000 50  0001 C CNN
@@
 AR Path="/5CD03534/5CD5414F/5CD65D2C" Ref="#PWR?"  Part="1"
 AR Path="/5CD47361/5CD5414F/5CD65D2C" Ref="#PWR?"  Part="1"
-AR Path="/5CF23C1A/5CD5414F/5CD65D2C" Ref="#PWR?"  Part="1"
-F 0 "#PWR?" H 3200 4250 50  0001 C CNN
+AR Path="/5CF23C1A/5CD5414F/5CD65D2C" Ref="#PWR051"  Part="1"
+F 0 "#PWR051" H 3200 4250 50  0001 C CNN
 F 1 "+5V" H 3250 4600 50  0000 C CNN
 F 2 "" H 3200 4400 50  0001 C CNN
@@
 AR Path="/5CD03534/5CD5414F/5CD6621A" Ref="C?"  Part="1"
 AR Path="/5CD47361/5CD5414F/5CD6621A" Ref="C?"  Part="1"
-AR Path="/5CF23C1A/5CD5414F/5CD6621A" Ref="C?"  Part="1"
-F 0 "C?" H 3100 4800 50  0000 R CNN
+AR Path="/5CF23C1A/5CD5414F/5CD6621A" Ref="C11"  Part="1"
+F 0 "C11" H 3100 4800 50  0000 R CNN
 F 1 "C106,0603" H 3100 4750 50  0000 R CNN
 F 2 "Capacitor_SMD:C_0603_1608Metric_Pad1.05x0.95mm_HandSolder" H 3200 4750 50  0001 C CNN
@@
 AR Path="/5CD03534/5CD5414F/5CD66224" Ref="C?"  Part="1"
 AR Path="/5CD47361/5CD5414F/5CD66224" Ref="C?"  Part="1"
-AR Path="/5CF23C1A/5CD5414F/5CD66224" Ref="C?"  Part="1"
-F 0 "C?" H 3550 4800 50  0000 L CNN
+AR Path="/5CF23C1A/5CD5414F/5CD66224" Ref="C12"  Part="1"
+F 0 "C12" H 3550 4800 50  0000 L CNN
 F 1 "C104,0603" H 3550 4750 50  0000 L CNN
 F 2 "Capacitor_SMD:C_0603_1608Metric_Pad1.05x0.95mm_HandSolder" H 3450 4750 50  0001 C CNN
@@
 AR Path="/5CD03534/5CD5414F/5CD68920" Ref="#PWR?"  Part="1"
 AR Path="/5CD47361/5CD5414F/5CD68920" Ref="#PWR?"  Part="1"
-AR Path="/5CF23C1A/5CD5414F/5CD68920" Ref="#PWR?"  Part="1"
-F 0 "#PWR?" H 3350 4800 50  0001 C CNN
+AR Path="/5CF23C1A/5CD5414F/5CD68920" Ref="#PWR052"  Part="1"
+F 0 "#PWR052" H 3350 4800 50  0001 C CNN
 F 1 "GND" H 3400 4850 50  0000 C CNN
 F 2 "" H 3350 5050 50  0001 C CNN
@@
 AR Path="/5CD03534/5CD5414F/5CD7BF83" Ref="Q?"  Part="1"
 AR Path="/5CD47361/5CD5414F/5CD7BF83" Ref="Q?"  Part="1"
-AR Path="/5CF23C1A/5CD5414F/5CD7BF83" Ref="Q?"  Part="1"
-F 0 "Q?" H 8850 3700 50  0000 L CNN
+AR Path="/5CF23C1A/5CD5414F/5CD7BF83" Ref="Q1"  Part="1"
+F 0 "Q1" H 8850 3700 50  0000 L CNN
 F 1 "SS9013_J3" H 8850 3650 50  0000 L CNN
 F 2 "footprint-lib:9013,J3,SOT23" H 8850 3575 50  0001 L CIN
@@
 AR Path="/5CD03534/5CD5414F/5CD7C99C" Ref="Q?"  Part="1"
 AR Path="/5CD47361/5CD5414F/5CD7C99C" Ref="Q?"  Part="1"
-AR Path="/5CF23C1A/5CD5414F/5CD7C99C" Ref="Q?"  Part="1"
-F 0 "Q?" H 8850 4350 50  0000 L CNN
+AR Path="/5CF23C1A/5CD5414F/5CD7C99C" Ref="Q2"  Part="1"
+F 0 "Q2" H 8850 4350 50  0000 L CNN
 F 1 "SS9013_J3" H 8850 4400 50  0000 L CNN
 F 2 "footprint-lib:9013,J3,SOT23" H 8850 4325 50  0001 L CIN
@@
 AR Path="/5CD03534/5CD5414F/5CD7F8D4" Ref="R?"  Part="1"
 AR Path="/5CD47361/5CD5414F/5CD7F8D4" Ref="R?"  Part="1"
-AR Path="/5CF23C1A/5CD5414F/5CD7F8D4" Ref="R?"  Part="1"
-F 0 "R?" V 8850 3650 50  0000 C CNN
+AR Path="/5CF23C1A/5CD5414F/5CD7F8D4" Ref="R16"  Part="1"
+F 0 "R16" V 8850 3650 50  0000 C CNN
 F 1 "R123,0603" V 8950 3650 50  0000 C CNN
 F 2 "Resistor_SMD:R_0603_1608Metric_Pad1.05x0.95mm_HandSolder" H 9100 3650 50  0001 C CNN
@@
 AR Path="/5CD03534/5CD5414F/5CD7FB22" Ref="R?"  Part="1"
 AR Path="/5CD47361/5CD5414F/5CD7FB22" Ref="R?"  Part="1"
-AR Path="/5CF23C1A/5CD5414F/5CD7FB22" Ref="R?"  Part="1"
-F 0 "R?" V 8850 4400 50  0000 C CNN
+AR Path="/5CF23C1A/5CD5414F/5CD7FB22" Ref="R17"  Part="1"
+F 0 "R17" V 8850 4400 50  0000 C CNN
 F 1 "R123,0603" V 8950 4400 50  0000 C CNN
 F 2 "Resistor_SMD:R_0603_1608Metric_Pad1.05x0.95mm_HandSolder" H 9100 4400 50  0001 C CNN
@@
 AR Path="/5CD03534/5CD5414F/5CD48A65" Ref="#PWR?"  Part="1"
 AR Path="/5CD47361/5CD5414F/5CD48A65" Ref="#PWR?"  Part="1"
-AR Path="/5CF23C1A/5CD5414F/5CD48A65" Ref="#PWR?"  Part="1"
-F 0 "#PWR?" H 7550 2250 50  0001 C CNN
+AR Path="/5CF23C1A/5CD5414F/5CD48A65" Ref="#PWR047"  Part="1"
+F 0 "#PWR047" H 7550 2250 50  0001 C CNN
 F 1 "GND" H 7600 2300 50  0000 C CNN
 F 2 "" H 7550 2500 50  0001 C CNN
@@
 AR Path="/5CD03534/5CD5414F/5CD693FB" Ref="#PWR?"  Part="1"
 AR Path="/5CD47361/5CD5414F/5CD693FB" Ref="#PWR?"  Part="1"
-AR Path="/5CF23C1A/5CD5414F/5CD693FB" Ref="#PWR?"  Part="1"
-F 0 "#PWR?" H 7250 1350 50  0001 C CNN
+AR Path="/5CF23C1A/5CD5414F/5CD693FB" Ref="#PWR046"  Part="1"
+F 0 "#PWR046" H 7250 1350 50  0001 C CNN
 F 1 "+5V" H 7300 1650 50  0000 C CNN
 F 2 "" H 7250 1500 50  0001 C CNN
@@
 	1300 1750 1650 1750
 $Comp
-L taobao-components:USB_Micro U?
+L taobao-components:USB_Micro U6
 U 1 1 5CF7C60C
 P 8050 1900
-F 0 "U?" H 8050 2365 50  0000 C CNN
+F 0 "U6" H 8050 2365 50  0000 C CNN
 F 1 "USB_Micro" H 8050 2274 50  0000 C CNN
 F 2 "footprint-lib:USB_Micro-B_Molex-105017-0001" H 8050 1400 50  0001 C CNN
@@
 AR Path="/5CD03534/5CD5414F/5CF81EDB" Ref="#PWR?"  Part="1"
 AR Path="/5CD47361/5CD5414F/5CF81EDB" Ref="#PWR?"  Part="1"
-AR Path="/5CF23C1A/5CD5414F/5CF81EDB" Ref="#PWR?"  Part="1"
-F 0 "#PWR?" H 8650 2250 50  0001 C CNN
+AR Path="/5CF23C1A/5CD5414F/5CF81EDB" Ref="#PWR048"  Part="1"
+F 0 "#PWR048" H 8650 2250 50  0001 C CNN
 F 1 "GND" H 8700 2300 50  0000 C CNN
 F 2 "" H 8650 2500 50  0001 C CNN
@@
 NoConn ~ 3800 4000
 NoConn ~ 4000 4450
+NoConn ~ 4250 1550
+NoConn ~ 3850 1550
+NoConn ~ 2300 2700
+NoConn ~ 2300 2800
+NoConn ~ 7250 2000
 $EndSCHEMATC

Commit message: after routing,
Parts:
- U7: footprint w_smd_qfn:qfn-28 -> footprint-lib:CP2102_qfn28
Changed lines of the file:
@@
 F 0 "U7" H 5050 3050 50  0000 L CNN
 F 1 "CP2102" H 5050 3000 50  0000 L CNN
-F 2 "w_smd_qfn:qfn-28" H 4000 1600 50  0001 C CNN
+F 2 "footprint-lib:CP2102_qfn28" H 4000 1600 50  0001 C CNN
 F 3 "" H 3500 3100 50  0001 C CNN
 	1    4000 3000
