File: hardware/ESP12_button.sch (KiCad schematic (older format))
At the start: 7 parts

Commit message: after DRC,
Parts:
- gave numbers to parts that had none: 7
Changed lines of the file:
@@
 AR Path="/5CD03534/5CD6BE5F/5CD6EFDD" Ref="#PWR?"  Part="1"
 AR Path="/5CD47361/5CD6BE5F/5CD6EFDD" Ref="#PWR?"  Part="1"
-AR Path="/5CF23C1A/5CD6BE5F/5CD6EFDD" Ref="#PWR?"  Part="1"
-F 0 "#PWR?" H 4050 1050 50  0001 C CNN
+AR Path="/5CF23C1A/5CD6BE5F/5CD6EFDD" Ref="#PWR053"  Part="1"
+F 0 "#PWR053" H 4050 1050 50  0001 C CNN
 F 1 "+3V3" H 4100 1400 50  0000 C CNN
 F 2 "" H 4050 1200 50  0001 C CNN
@@
 AR Path="/5CD03534/5CD6BE5F/5CD6F2CA" Ref="R?"  Part="1"
 AR Path="/5CD47361/5CD6BE5F/5CD6F2CA" Ref="R?"  Part="1"
-AR Path="/5CF23C1A/5CD6BE5F/5CD6F2CA" Ref="R?"  Part="1"
-F 0 "R?" H 4150 1550 50  0000 L CNN
+AR Path="/5CF23C1A/5CD6BE5F/5CD6F2CA" Ref="R18"  Part="1"
+F 0 "R18" H 4150 1550 50  0000 L CNN
 F 1 "R471,0603" H 4150 1500 50  0000 L CNN
 F 2 "Resistor_SMD:R_0603_1608Metric_Pad1.05x0.95mm_HandSolder" H 4050 1500 50  0001 C CNN
@@
 AR Path="/5CD03534/5CD6BE5F/5CD6F699" Ref="D?"  Part="1"
 AR Path="/5CD47361/5CD6BE5F/5CD6F699" Ref="D?"  Part="1"
-AR Path="/5CF23C1A/5CD6BE5F/5CD6F699" Ref="D?"  Part="1"
-F 0 "D?" V 4100 1750 50  0000 R CNN
+AR Path="/5CF23C1A/5CD6BE5F/5CD6F699" Ref="D5"  Part="1"
+F 0 "D5" V 4100 1750 50  0000 R CNN
 F 1 "LED_BLUE,0603" V 4050 1750 50  0000 R CNN
 F 2 "LED_SMD:LED_0603_1608Metric_Pad1.05x0.95mm_HandSolder" V 4050 1850 50  0001 C CNN
@@
 AR Path="/5CD03534/5CD6BE5F/5CD70197" Ref="R?"  Part="1"
 AR Path="/5CD47361/5CD6BE5F/5CD70197" Ref="R?"  Part="1"
-AR Path="/5CF23C1A/5CD6BE5F/5CD70197" Ref="R?"  Part="1"
-F 0 "R?" H 4150 2300 50  0000 L CNN
+AR Path="/5CF23C1A/5CD6BE5F/5CD70197" Ref="R20"  Part="1"
+F 0 "R20" H 4150 2300 50  0000 L CNN
 F 1 "R0,0603" H 4150 2250 50  0000 L CNN
 F 2 "Resistor_SMD:R_0603_1608Metric_Pad1.05x0.95mm_HandSolder" H 4050 2250 50  0001 C CNN
@@
 AR Path="/5CD03534/5CD6BE5F/5CD705A6" Ref="SW?"  Part="1"
 AR Path="/5CD47361/5CD6BE5F/5CD705A6" Ref="SW?"  Part="1"
-AR Path="/5CF23C1A/5CD6BE5F/5CD705A6" Ref="SW?"  Part="1"
-F 0 "SW?" V 4300 2900 50  0000 L CNN
+AR Path="/5CF23C1A/5CD6BE5F/5CD705A6" Ref="SW2"  Part="1"
+F 0 "SW2" V 4300 2900 50  0000 L CNN
 F 1 "SW_RESET,2_leg,SMD" V 4350 2900 50  0000 L CNN
 F 2 "footprint-lib:SW_SPST_CK_RS282G05A3" H 4350 2950 50  0001 C CNN
@@
 AR Path="/5CD03534/5CD6BE5F/5CD70C90" Ref="R?"  Part="1"
 AR Path="/5CD47361/5CD6BE5F/5CD70C90" Ref="R?"  Part="1"
-AR Path="/5CF23C1A/5CD6BE5F/5CD70C90" Ref="R?"  Part="1"
-F 0 "R?" H 4700 2300 50  0000 L CNN
+AR Path="/5CF23C1A/5CD6BE5F/5CD70C90" Ref="R21"  Part="1"
+F 0 "R21" H 4700 2300 50  0000 L CNN
 F 1 "R471,0603" H 4700 2250 50  0000 L CNN
 F 2 "Resistor_SMD:R_0603_1608Metric_Pad1.05x0.95mm_HandSolder" H 4600 2250 50  0001 C CNN
@@
 AR Path="/5CD03534/5CD6BE5F/5CD72E50" Ref="#PWR?"  Part="1"
 AR Path="/5CD47361/5CD6BE5F/5CD72E50" Ref="#PWR?"  Part="1"
-AR Path="/5CF23C1A/5CD6BE5F/5CD72E50" Ref="#PWR?"  Part="1"
-F 0 "#PWR?" H 4350 2900 50  0001 C CNN
+AR Path="/5CF23C1A/5CD6BE5F/5CD72E50" Ref="#PWR055"  Part="1"
+F 0 "#PWR055" H 4350 2900 50  0001 C CNN
 F 1 "GND" H 4400 2950 50  0000 C CNN
 F 2 "" H 4350 3150 50  0001 C CNN
@@
 AR Path="/5CD03534/5CD6BE5F/5CD73ECF" Ref="SW?"  Part="1"
 AR Path="/5CD47361/5CD6BE5F/5CD73ECF" Ref="SW?"  Part="1"
-AR Path="/5CF23C1A/5CD6BE5F/5CD73ECF" Ref="SW?"  Part="1"
-F 0 "SW?" V 5700 2650 50  0000 L CNN
+AR Path="/5CF23C1A/5CD6BE5F/5CD73ECF" Ref="SW1"  Part="1"
+F 0 "SW1" V 5700 2650 50  0000 L CNN
 F 1 "FLASH_BUTTON" V 5750 2650 50  0000 L CNN
 F 2 "footprint-lib:SW_SPST_CK_RS282G05A3" H 5750 2700 50  0001 C CNN
@@
 AR Path="/5CD03534/5CD6BE5F/5CD7498A" Ref="R?"  Part="1"
 AR Path="/5CD47361/5CD6BE5F/5CD7498A" Ref="R?"  Part="1"
-AR Path="/5CF23C1A/5CD6BE5F/5CD7498A" Ref="R?"  Part="1"
-F 0 "R?" H 5850 2100 50  0000 L CNN
+AR Path="/5CF23C1A/5CD6BE5F/5CD7498A" Ref="R19"  Part="1"
+F 0 "R19" H 5850 2100 50  0000 L CNN
 F 1 "R471,0603" H 5850 2050 50  0000 L CNN
 F 2 "Resistor_SMD:R_0603_1608Metric_Pad1.05x0.95mm_HandSolder" H 5750 2050 50  0001 C CNN
@@
 AR Path="/5CD03534/5CD6BE5F/5CD75A97" Ref="#PWR?"  Part="1"
 AR Path="/5CD47361/5CD6BE5F/5CD75A97" Ref="#PWR?"  Part="1"
-AR Path="/5CF23C1A/5CD6BE5F/5CD75A97" Ref="#PWR?"  Part="1"
-F 0 "#PWR?" H 5750 2650 50  0001 C CNN
+AR Path="/5CF23C1A/5CD6BE5F/5CD75A97" Ref="#PWR054"  Part="1"
+F 0 "#PWR054" H 5750 2650 50  0001 C CNN
 F 1 "GND" H 5800 2700 50  0000 C CNN
 F 2 "" H 5750 2900 50  0001 C CNN

Commit message: update for RESET BUTTON,
Parts:
- SW1: value FLASH_BUTTON -> FLASH
- SW2: value SW_RESET,2_leg,SMD -> RST
Changed lines of the file:
@@
 AR Path="/5CF23C1A/5CD6BE5F/5CD705A6" Ref="SW2"  Part="1"
 F 0 "SW2" V 4300 2900 50  0000 L CNN
-F 1 "SW_RESET,2_leg,SMD" V 4350 2900 50  0000 L CNN
+F 1 "RST" V 4350 2900 50  0000 L CNN
 F 2 "footprint-lib:SW_SPST_CK_RS282G05A3" H 4350 2950 50  0001 C CNN
 F 3 "~" H 4350 2950 50  0001 C CNN
@@
 AR Path="/5CF23C1A/5CD6BE5F/5CD73ECF" Ref="SW1"  Part="1"
 F 0 "SW1" V 5700 2650 50  0000 L CNN
-F 1 "FLASH_BUTTON" V 5750 2650 50  0000 L CNN
+F 1 "FLASH" V 5750 2650 50  0000 L CNN
 F 2 "footprint-lib:SW_SPST_CK_RS282G05A3" H 5750 2700 50  0001 C CNN
 F 3 "~" H 5750 2700 50  0001 C CNN
